Commit message: asd

File: assets/urdf/tatbot.urdf (robot description, URDF)
Before this commit: robot mobile_ai, 61 links, 60 joints
Links:
- added link 300mm_left_rail_left; visual mesh filename=meshes/frame/t2020_300mm.stl scale=0.001 0.001 0.001
- added link 300mm_left_rail_right; visual mesh filename=meshes/frame/t2020_300mm.stl scale=0.001 0.001 0.001
- added link 300mm_right_rail_left; visual mesh filename=meshes/frame/t2020_300mm.stl scale=0.001 0.001 0.001
- added link 300mm_right_rail_right; visual mesh filename=meshes/frame/t2020_300mm.stl scale=0.001 0.001 0.001
- added link 300mm_vertical_top; visual mesh filename=meshes/frame/t2020_300mm.stl scale=0.001 0.001 0.001
- added link 600mm_back_horizontal; visual mesh filename=meshes/frame/t2020_600mm.stl scale=0.001 0.001 0.001
- added link 600mm_front_horizontal; visual mesh filename=meshes/frame/t2020_600mm.stl scale=0.001 0.001 0.001
- added link 600mm_vertical_left; visual mesh filename=meshes/frame/t2020_600mm.stl scale=0.001 0.001 0.001
- added link 600mm_vertical_right; visual mesh filename=meshes/frame/t2020_600mm.stl scale=0.001 0.001 0.001
Joints:
- added joint 300mm_left_rail_left_joint: type fixed, parent root, child 300mm_left_rail_left, origin xyz=-0.12 0.258125 -0.01 rpy=0 0 0
- added joint 300mm_left_rail_right_joint: type fixed, parent root, child 300mm_left_rail_right, origin xyz=-0.12 0.218125 -0.01 rpy=0 0 0
- added joint 300mm_right_rail_left_joint: type fixed, parent root, child 300mm_right_rail_left, origin xyz=-0.12 -0.218125 -0.01 rpy=0 0 0
- added joint 300mm_right_rail_right_joint: type fixed, parent root, child 300mm_right_rail_right, origin xyz=-0.12 -0.258125 -0.01 rpy=0 0 0
- added joint 300mm_vertical_top_joint: type fixed, parent root, child 300mm_vertical_top, origin xyz=-0.267 0 0.59 rpy=0 0 0
- added joint 600mm_back_horizontal_joint: type fixed, parent root, child 600mm_back_horizontal, origin xyz=-0.267 0 -0.03 rpy=0 0 0
- added joint 600mm_front_horizontal_joint: type fixed, parent root, child 600mm_front_horizontal, origin xyz=0.0278 0 -0.03 rpy=0 0 0
- added joint 600mm_vertical_left_joint: type fixed, parent root, child 600mm_vertical_left, origin xyz=-0.267 0.08128 0.28 rpy=0 0 0
- added joint 600mm_vertical_right_joint: type fixed, parent root, child 600mm_vertical_right, origin xyz=-0.267 -0.08128 0.28 rpy=0 0 0
- joint camera1_mount_joint: origin xyz=-0.3 -0.22 0.4 rpy=0 1.5707963267948966 0 -> xyz=0.08 0.258125 -0.05 rpy=0 1.5707963267948966 0
- joint camera5_mount_joint: origin xyz=0 -0.2 0.5 rpy=0 1.5707963267948966 0 -> xyz=0.08 -0.258125 -0.05 rpy=0 1.5707963267948966 0
- joint left/mount_joint: origin xyz=-0.20 0 0 rpy=0 0 0 -> xyz=0 0.238125 0 rpy=0 0 0
- joint right/mount_joint: origin xyz=0 -0.2413 0 rpy=0 0 0 -> xyz=0 -0.238125 0 rpy=0 0 0

Commit message: asd

File: assets/urdf/tatbot.urdf (robot description, URDF)
Before this commit: robot mobile_ai, 70 links, 69 joints
Joints:
- joint cam_high_joint: origin xyz=0.12 -0.30 0.6 rpy=0 1.5707963267948966 0 -> xyz=-0.24 0 0.64 rpy=0 0.7853981633974483 0
- joint camera1_mount_joint: origin xyz=0.08 0.258125 -0.05 rpy=0 1.5707963267948966 0 -> xyz=0.0378 0.258125 -0.08 rpy=0 1.5707963267948966 0
- joint camera2_mount_joint: origin xyz=0 0.2 0.5 rpy=0 1.5707963267948966 0 -> xyz=-0.257 0.08128 0.5 rpy=0 1.5707963267948966 0
- joint camera3_mount_joint: origin xyz=0 0.1 0.7 rpy=0 1.5707963267948966 0 -> xyz=-0.257 0.06 0.7 rpy=0 1.5707963267948966 0
- joint camera4_mount_joint: origin xyz=0 -0.1 0.7 rpy=0 1.5707963267948966 0 -> xyz=-0.257 -0.06 0.7 rpy=0 1.5707963267948966 0
- joint camera5_mount_joint: origin xyz=0.08 -0.258125 -0.05 rpy=0 1.5707963267948966 0 -> xyz=0.0378 -0.258125 -0.08 rpy=0 1.5707963267948966 0

Commit message: asd

File: assets/urdf/tatbot.urdf (robot description, URDF)
Before this commit: robot mobile_ai, 70 links, 69 joints
Joints:
- joint cam_high_joint: origin xyz=-0.24 0 0.64 rpy=0 0.7853981633974483 0 -> xyz=-0.22 0 0.63 rpy=0 0.7853981633974483 0
- joint left/mount_joint: origin xyz=0 0.238125 0 rpy=0 0 0 -> xyz=0 0.238125 0 rpy=0 0 -1.57079632679
- joint right/mount_joint: origin xyz=0 -0.238125 0 rpy=0 0 0 -> xyz=0 -0.238125 0 rpy=0 0 -1.57079632679

Commit message: asd

File: assets/urdf/tatbot.urdf (robot description, URDF)
Before this commit: robot mobile_ai, 70 links, 69 joints
Joints:
- joint right/mount_joint: origin xyz=0 -0.238125 0 rpy=0 0 -1.57079632679 -> xyz=0 -0.238125 0 rpy=0 0 0

Commit message: asd

File: assets/urdf/tatbot.urdf (robot description, URDF)
Before this commit: robot mobile_ai, 70 links, 69 joints
Joints:
- joint left/mount_joint: origin xyz=0 0.238125 0 rpy=0 0 -1.57079632679 -> xyz=0 0.238125 0 rpy=0 0 0

Commit message: asd

File: assets/urdf/tatbot.urdf (robot description, URDF)
Before this commit: robot mobile_ai, 70 links, 69 joints
Links:
- removed link right/gripper_left
- removed link right/gripper_right
Joints:
- removed joint right/left_gripper_joint

Commit message: asd

File: assets/urdf/tatbot.urdf (robot description, URDF)
Before this commit: robot mobile_ai, 68 links, 68 joints
Links:
- removed link cam_high_bottom_screw_frame
- removed link cam_high_color_frame
- removed link cam_high_color_optical_frame
- removed link cam_high_depth_frame
- removed link cam_high_depth_optical_frame
- removed link cam_high_infra1_frame
- removed link cam_high_infra1_optical_frame
- removed link cam_high_infra2_frame
- removed link cam_high_infra2_optical_frame
- removed link cam_high_link
- removed link right/camera_bottom_screw_frame
- removed link right/camera_color_frame
- removed link right/camera_color_optical_frame
- removed link right/camera_depth_frame
- removed link right/camera_depth_optical_frame
- removed link right/camera_infra1_frame
- removed link right/camera_infra1_optical_frame
- removed link right/camera_infra2_frame
- removed link right/camera_infra2_optical_frame
- removed link right/camera_link
- removed link right/camera_mount_d405
- added link realsense1_bottom_screw_frame
- added link realsense1_color_frame
- added link realsense1_color_optical_frame
- added link realsense1_depth_frame
- added link realsense1_depth_optical_frame
- added link realsense1_infra1_frame
- added link realsense1_infra1_optical_frame
- added link realsense1_infra2_frame
- added link realsense1_infra2_optical_frame
- added link realsense1_link, mass 0.072; collision box size=0.023 0.042 0.042; visual mesh filename=meshes/cameras/d405.stl scale=0.001 0.001 0.001
- added link realsense2_bottom_screw_frame
- added link realsense2_color_frame
- added link realsense2_color_optical_frame
- added link realsense2_depth_frame
- added link realsense2_depth_optical_frame
- added link realsense2_infra1_frame
- added link realsense2_infra1_optical_frame
- added link realsense2_infra2_frame
- added link realsense2_infra2_optical_frame
- added link realsense2_link, mass 0.072; collision box size=0.023 0.042 0.042; visual mesh filename=meshes/cameras/d405.stl scale=0.001 0.001 0.001
Joints:
- removed joint cam_high_color_joint
- removed joint cam_high_color_optical_joint
- removed joint cam_high_depth_joint
- removed joint cam_high_depth_optical_joint
- removed joint cam_high_infra1_joint
- removed joint cam_high_infra1_optical_joint
- removed joint cam_high_infra2_joint
- removed joint cam_high_infra2_optical_joint
- removed joint cam_high_joint
- removed joint cam_high_link_joint
- removed joint right/camera_color_joint
- removed joint right/camera_color_optical_joint
- removed joint right/camera_depth_joint
- removed joint right/camera_depth_optical_joint
- removed joint right/camera_infra1_joint
- removed joint right/camera_infra1_optical_joint
- removed joint right/camera_infra2_joint
- removed joint right/camera_infra2_optical_joint
- removed joint right/camera_joint
- removed joint right/camera_link_joint
- removed joint right/camera_mount_joint
- added joint realsense1_color_joint: type fixed, parent realsense1_link, child realsense1_color_frame, origin xyz=0 0.0 0 rpy=0 0 0
- added joint realsense1_color_optical_joint: type fixed, parent realsense1_color_frame, child realsense1_color_optical_frame, origin xyz=0 0 0 rpy=-1.5707963267948966 0 -1.5707963267948966
- added joint realsense1_depth_joint: type fixed, parent realsense1_link, child realsense1_depth_frame, origin xyz=0 0 0 rpy=0 0 0
- added joint realsense1_depth_optical_joint: type fixed, parent realsense1_depth_frame, child realsense1_depth_optical_frame, origin xyz=0 0 0 rpy=-1.5707963267948966 0 -1.5707963267948966
- added joint realsense1_infra1_joint: type fixed, parent realsense1_link, child realsense1_infra1_frame, origin xyz=0 0.0 0 rpy=0 0 0
- added joint realsense1_infra1_optical_joint: type fixed, parent realsense1_infra1_frame, child realsense1_infra1_optical_frame, origin xyz=0 0 0 rpy=-1.5707963267948966 0 -1.5707963267948966
- added joint realsense1_infra2_joint: type fixed, parent realsense1_link, child realsense1_infra2_frame, origin xyz=0 -0.018 0 rpy=0 0 0
- added joint realsense1_infra2_optical_joint: type fixed, parent realsense1_infra2_frame, child realsense1_infra2_optical_frame, origin xyz=0 0 0 rpy=-1.5707963267948966 0 -1.5707963267948966
- added joint realsense1_joint: type fixed, parent root, child realsense1_bottom_screw_frame, origin xyz=-0.22 0 0.63 rpy=0 0.7853981633974483 0
- added joint realsense1_link_joint: type fixed, parent realsense1_bottom_screw_frame, child realsense1_link, origin xyz=0.01085 0.009 0.021 rpy=0 0 0
- added joint realsense2_color_joint: type fixed, parent realsense2_link, child realsense2_color_frame, origin xyz=0 0.0 0 rpy=0 0 0
- added joint realsense2_color_optical_joint: type fixed, parent realsense2_color_frame, child realsense2_color_optical_frame, origin xyz=0 0 0 rpy=-1.5707963267948966 0 -1.5707963267948966
- added joint realsense2_depth_joint: type fixed, parent realsense2_link, child realsense2_depth_frame, origin xyz=0 0 0 rpy=0 0 0
- added joint realsense2_depth_optical_joint: type fixed, parent realsense2_depth_frame, child realsense2_depth_optical_frame, origin xyz=0 0 0 rpy=-1.5707963267948966 0 -1.5707963267948966
- added joint realsense2_infra1_joint: type fixed, parent realsense2_link, child realsense2_infra1_frame, origin xyz=0 0.0 0 rpy=0 0 0
- added joint realsense2_infra1_optical_joint: type fixed, parent realsense2_infra1_frame, child realsense2_infra1_optical_frame, origin xyz=0 0 0 rpy=-1.5707963267948966 0 -1.5707963267948966
- added joint realsense2_infra2_joint: type fixed, parent realsense2_link, child realsense2_infra2_frame, origin xyz=0 -0.018 0 rpy=0 0 0
- added joint realsense2_infra2_optical_joint: type fixed, parent realsense2_infra2_frame, child realsense2_infra2_optical_frame, origin xyz=0 0 0 rpy=-1.5707963267948966 0 -1.5707963267948966
- added joint realsense2_joint: type fixed, parent root, child realsense2_bottom_screw_frame, origin xyz=-0.22 0.1 0.63 rpy=0 0.7853981633974483 0
- added joint realsense2_link_joint: type fixed, parent realsense2_bottom_screw_frame, child realsense2_link, origin xyz=0.01085 0.009 0.021 rpy=0 0 0

Commit message: asd

File: assets/urdf/tatbot.urdf (robot description, URDF)
Before this commit: robot mobile_ai, 67 links, 67 joints
Links:
- removed link right/ee_gripper_link
- added link right/leader_finger_right_thumb, mass 0.02088075; collision mesh filename=meshes/wxai/leader_finger_right_thumb.stl; visual mesh filename=meshes/wxai/leader_finger_right_thumb.stl
- added link right/tattoo_needle; collision cylinder length=0.035 radius=0.002; visual cylinder length=0.035 radius=0.002
- added link right/tattoo_pen, mass 0.01; collision cylinder length=0.1 radius=0.012; visual cylinder length=0.1 radius=0.012
Joints:
- removed joint right/ee_gripper
- removed joint right/right_gripper_joint
- added joint right/right_index_joint: type fixed, parent right/carriage_right, child right/leader_finger_right_thumb, origin xyz=0 0 0 rpy=0 0 0, axis 0 0 0
- added joint right/tattoo_needle_joint: type fixed, parent right/tattoo_pen, child right/tattoo_needle, origin xyz=0.035 0 0 rpy=0 0 0
- added joint right/tattoo_pen_joint: type fixed, parent right/leader_finger_right_thumb, child right/tattoo_pen, origin xyz=0.1 -0.01 0.055 rpy=0 0 0

Commit message: asd

File: assets/urdf/tatbot.urdf (robot description, URDF)
Before this commit: robot tatbot, 69 links, 68 joints
Joints:
- joint right/tattoo_pen_joint: origin xyz=0.1 -0.01 0.055 rpy=0 0 0 -> xyz=0.1 0.01 0.055 rpy=0 0 0

Commit message: asd

File: assets/urdf/tatbot.urdf (robot description, URDF)
Before this commit: robot tatbot, 69 links, 68 joints
Joints:
- joint realsense1_joint: origin xyz=-0.22 0 0.63 rpy=0 0.7853981633974483 0 -> xyz=-0.22 0 0.2 rpy=0 0.7853981633974483 0
- joint realsense2_joint: origin xyz=-0.22 0.1 0.63 rpy=0 0.7853981633974483 0 -> xyz=0.2 -0.15 0.05 rpy=0 0.7853981633974483 2.3

Commit message: asd

File: assets/urdf/tatbot.urdf (robot description, URDF)
Before this commit: robot tatbot, 69 links, 68 joints
Joints:
- joint right/right_index_joint: origin xyz=0 0 0 rpy=0 0 0 -> xyz=0 0 -0.008 rpy=0 0 0

Commit message: tags, inkpalette in urdf

File: assets/urdf/tatbot.urdf (robot description, URDF)
Before this commit: robot tatbot, 69 links, 68 joints
Links:
- added link inkpalette
- added link inkpalette_mesh; visual mesh filename=meshes/inkpalette/inkpalette.obj scale=1 1 1
- added link tag6; visual mesh filename=meshes/tags/16h5_006/tag.obj scale=1 1 1
Joints:
- added joint inkpalette_joint: type fixed, parent root, child inkpalette, origin xyz=-0.08 0 0 rpy=0 0 1.57
- added joint inkpalette_mesh_joint: type fixed, parent inkpalette, child inkpalette_mesh, origin xyz=0 0 0 rpy=0 0 0
- added joint tag6_joint: type fixed, parent root, child tag6, origin xyz=0 0 0 rpy=0 0 0

Commit message: skin mesh, more tags

File: assets/urdf/tatbot.urdf (robot description, URDF)
Before this commit: robot tatbot, 72 links, 71 joints
Links:
- added link inkcap_large
- added link inkcap_medium_1
- added link inkcap_medium_2
- added link inkcap_small_1
- added link inkcap_small_2
- added link inkcap_small_3
- added link skin
- added link skin_mesh; visual mesh filename=meshes/skin/skin.obj scale=1 1 1
- added link tag10; visual mesh filename=meshes/tags/16h5_010/tag.obj scale=1 1 1
- added link tag11; visual mesh filename=meshes/tags/16h5_011/tag.obj scale=1 1 1
- added link tag7; visual mesh filename=meshes/tags/16h5_007/tag.obj scale=1 1 1
- added link tag9; visual mesh filename=meshes/tags/16h5_009/tag.obj scale=1 1 1
Joints:
- removed joint inkpalette_joint
- added joint inkcap_large_joint: type fixed, parent inkpalette, child inkcap_large, origin xyz=0 0 0 rpy=0 0 0
- added joint inkcap_medium_1_joint: type fixed, parent inkpalette, child inkcap_medium_1, origin xyz=0 0 0 rpy=0 0 0
- added joint inkcap_medium_2_joint: type fixed, parent inkpalette, child inkcap_medium_2, origin xyz=0 0 0 rpy=0 0 0
- added joint inkcap_small_1_joint: type fixed, parent inkpalette, child inkcap_small_1, origin xyz=0 0 0 rpy=0 0 0
- added joint inkcap_small_2_joint: type fixed, parent inkpalette, child inkcap_small_2, origin xyz=0 0 0 rpy=0 0 0
- added joint inkcap_small_3_joint: type fixed, parent inkpalette, child inkcap_small_3, origin xyz=0 0 0 rpy=0 0 0
- added joint skin_mesh_joint: type fixed, parent skin, child skin_mesh, origin xyz=0 0 0 rpy=0 0 0
- added joint tag10_joint: type fixed, parent root, child tag10, origin xyz=0 0 0.01 rpy=0 0 0
- added joint tag11_joint: type fixed, parent root, child tag11, origin xyz=0.2 0 0.01 rpy=0 0 0
- added joint tag7_joint: type fixed, parent right/leader_finger_right_thumb, child tag7, origin xyz=0.002 0 0 rpy=0 1.5707963267948966 0
- added joint tag9_joint: type fixed, parent root, child tag9, origin xyz=-0.05 0 0.01 rpy=0 0 0
- added joint tag_to_inkpalette_joint: type fixed, parent tag9, child inkpalette, origin xyz=-0.04 0 -0.01 rpy=0 0 1.57
- added joint tag_to_skin_joint: type fixed, parent tag11, child skin, origin xyz=-0.06 0.04 -0.02 rpy=0 0 0
- joint tag6_joint: origin xyz=0 0 0 rpy=0 0 0 -> xyz=0.002 0 0 rpy=0 1.5707963267948966 0; parent root -> left/leader_finger_left_thumb

Commit message: asd

File: assets/urdf/tatbot.urdf (robot description, URDF)
Before this commit: robot tatbot, 84 links, 83 joints
Links:
- removed link inkpalette
Joints:
- removed joint tag_to_inkpalette_joint
- joint inkcap_large_joint: origin xyz=0 0 0 rpy=0 0 0 -> xyz=-0.002 0.059 0 rpy=0 0 0; parent inkpalette -> tag9
- joint inkcap_medium_1_joint: origin xyz=0 0 0 rpy=0 0 0 -> xyz=-0.02 0.048 0 rpy=0 0 0; parent inkpalette -> tag9
- joint inkcap_medium_2_joint: origin xyz=0 0 0 rpy=0 0 0 -> xyz=-0.032 0.06 0 rpy=0 0 0; parent inkpalette -> tag9
- joint inkcap_small_1_joint: origin xyz=0 0 0 rpy=0 0 0 -> xyz=0.007 0.045 0 rpy=0 0 0; parent inkpalette -> tag9
- joint inkcap_small_2_joint: origin xyz=0 0 0 rpy=0 0 0 -> xyz=-0.012 0.074 0 rpy=0 0 0; parent inkpalette -> tag9
- joint inkcap_small_3_joint: origin xyz=0 0 0 rpy=0 0 0 -> xyz=-0.025 0.082 0 rpy=0 0 0; parent inkpalette -> tag9
- joint inkpalette_mesh_joint: parent inkpalette -> tag9

Commit message: Update URDF to include inkpalette and adjust joint parents; refactor tag tracking in _tag.py and bot_scan.py for improved detection and image processing.

File: assets/urdf/tatbot.urdf (robot description, URDF)
Before this commit: robot tatbot, 83 links, 82 joints
Links:
- added link inkpalette
Joints:
- added joint tag_to_inkpalette_joint: type fixed, parent tag9, child inkpalette, origin xyz=0 0 0 rpy=0 0 0
- joint inkcap_large_joint: parent tag9 -> inkpalette
- joint inkcap_medium_1_joint: parent tag9 -> inkpalette
- joint inkcap_medium_2_joint: parent tag9 -> inkpalette
- joint inkcap_small_1_joint: parent tag9 -> inkpalette
- joint inkcap_small_2_joint: parent tag9 -> inkpalette
- joint inkcap_small_3_joint: parent tag9 -> inkpalette
- joint inkpalette_mesh_joint: parent tag9 -> inkpalette

Commit message: asd

File: assets/urdf/tatbot.urdf (robot description, URDF)
Before this commit: robot tatbot, 84 links, 83 joints
Joints:
- joint tag9_joint: origin xyz=-0.05 0 0.01 rpy=0 0 0 -> xyz=-0.09 0 0.01 rpy=0 0 0

Commit message: HACK make carriage joints smol

File: assets/urdf/tatbot.urdf (robot description, URDF)
Before this commit: robot tatbot, 84 links, 83 joints
Joints:
- joint left/left_carriage_joint: limit lower=0.0 upper=0.044 effort=400.0 velocity=0.0875 -> lower=0.0 upper=0.001 effort=400.0 velocity=0.0875
- joint left/right_carriage_joint: limit lower=0.0 upper=0.044 effort=400.0 velocity=0.0875 -> lower=0.0 upper=0.001 effort=400.0 velocity=0.0875
- joint right/left_carriage_joint: limit lower=0.0 upper=0.044 effort=400.0 velocity=0.0875 -> lower=0.0 upper=0.001 effort=400.0 velocity=0.0875
- joint right/right_carriage_joint: limit lower=0.0 upper=0.044 effort=400.0 velocity=0.0875 -> lower=0.0 upper=0.001 effort=400.0 velocity=0.0875

Commit message: asd

File: assets/urdf/tatbot.urdf (robot description, URDF)
Before this commit: robot tatbot, 84 links, 83 joints
Joints:
- joint tag11_joint: origin xyz=0.2 0 0.01 rpy=0 0 0 -> xyz=0.2 0 -0.01 rpy=0 0 0
- joint tag9_joint: origin xyz=-0.09 0 0.01 rpy=0 0 0 -> xyz=-0.09 0 0.0 rpy=0 0 0

Commit message: asd

File: assets/urdf/tatbot.urdf (robot description, URDF)
Before this commit: robot tatbot, 84 links, 83 joints
Joints:
- joint tag11_joint: origin xyz=0.2 0 -0.01 rpy=0 0 0 -> xyz=0.25 -0.05 -0.01 rpy=0 0 0

Commit message: new palette

File: assets/urdf/tatbot.urdf (robot description, URDF)
Before this commit: robot tatbot, 84 links, 83 joints
Links:
- removed link skin
- removed link skin_mesh
- removed link tag10
- removed link tag11
- removed link tag9
- added link tag0; visual mesh filename=meshes/tags/16h5_009/tag.obj scale=1 1 1
- added link tag1; visual mesh filename=meshes/tags/16h5_009/tag.obj scale=1 1 1
- added link tag2; visual mesh filename=meshes/tags/16h5_009/tag.obj scale=1 1 1
Joints:
- removed joint skin_mesh_joint
- removed joint tag10_joint
- removed joint tag11_joint
- removed joint tag9_joint
- removed joint tag_to_inkpalette_joint
- removed joint tag_to_skin_joint
- added joint inkpalette_joint: type fixed, parent root, child inkpalette, origin xyz=0 0 0 rpy=0 0 0
- added joint tag0_joint: type fixed, parent root, child tag0, origin xyz=0 0 0.01 rpy=0 0 0
- added joint tag1_joint: type fixed, parent root, child tag1, origin xyz=0 0 0.01 rpy=0 0 0
- added joint tag2_joint: type fixed, parent root, child tag2, origin xyz=0 0 0.01 rpy=0 0 0
