Commit message: inkcaps

File: urdf/tatbot.urdf (robot description, URDF)
Before this commit: robot tatbot, 82 links, 81 joints
Links:
- removed link inkcap_large
- removed link inkcap_medium_1
- removed link inkcap_medium_2
- removed link inkcap_small_1
- removed link inkcap_small_2
- removed link inkcap_small_3
- added link inkcap_left_large
- added link inkcap_left_medium_1
- added link inkcap_left_medium_2
- added link inkcap_left_small_1
- added link inkcap_left_small_2
- added link inkcap_left_small_3
- added link inkcap_right_large
- added link inkcap_right_medium_0
- added link inkcap_right_medium_1
- added link inkcap_right_medium_2
- added link inkcap_right_small_0
- added link inkcap_right_small_1
- added link inkcap_right_small_2
- added link inkcap_right_small_3
Joints:
- removed joint inkcap_large_joint
- removed joint inkcap_medium_1_joint
- removed joint inkcap_medium_2_joint
- removed joint inkcap_small_1_joint
- removed joint inkcap_small_2_joint
- removed joint inkcap_small_3_joint
- added joint inkcap_left_large_joint: type fixed, parent inkpalette, child inkcap_left_large, origin xyz=-0.002 0.059 0 rpy=0 0 0
- added joint inkcap_left_medium_1_joint: type fixed, parent inkpalette, child inkcap_left_medium_1, origin xyz=-0.02 0.048 0 rpy=0 0 0
- added joint inkcap_left_medium_2_joint: type fixed, parent inkpalette, child inkcap_left_medium_2, origin xyz=-0.032 0.06 0 rpy=0 0 0
- added joint inkcap_left_small_1_joint: type fixed, parent inkpalette, child inkcap_left_small_1, origin xyz=0.007 0.045 0 rpy=0 0 0
- added joint inkcap_left_small_2_joint: type fixed, parent inkpalette, child inkcap_left_small_2, origin xyz=-0.012 0.074 0 rpy=0 0 0
- added joint inkcap_left_small_3_joint: type fixed, parent inkpalette, child inkcap_left_small_3, origin xyz=-0.025 0.082 0 rpy=0 0 0
- added joint inkcap_right_large_joint: type fixed, parent inkpalette, child inkcap_right_large, origin xyz=0.002 -0.059 0 rpy=0 0 0
- added joint inkcap_right_medium_0_joint: type fixed, parent inkpalette, child inkcap_right_medium_0, origin xyz=0.02 -0.048 0 rpy=0 0 0
- added joint inkcap_right_medium_1_joint: type fixed, parent inkpalette, child inkcap_right_medium_1, origin xyz=0.032 -0.06 0 rpy=0 0 0
- added joint inkcap_right_medium_2_joint: type fixed, parent inkpalette, child inkcap_right_medium_2, origin xyz=0.015 -0.07 0 rpy=0 0 0
- added joint inkcap_right_small_0_joint: type fixed, parent inkpalette, child inkcap_right_small_0, origin xyz=-0.007 -0.045 0 rpy=0 0 0
- added joint inkcap_right_small_1_joint: type fixed, parent inkpalette, child inkcap_right_small_1, origin xyz=0.012 -0.074 0 rpy=0 0 0
- added joint inkcap_right_small_2_joint: type fixed, parent inkpalette, child inkcap_right_small_2, origin xyz=0.025 -0.082 0 rpy=0 0 0
- added joint inkcap_right_small_3_joint: type fixed, parent inkpalette, child inkcap_right_small_3, origin xyz=0.018 -0.065 0 rpy=0 0 0

Commit message: asd

File: urdf/tatbot.urdf (robot description, URDF)
Before this commit: robot tatbot, 90 links, 89 joints
Links:
- removed link inkpalette
- removed link inkpalette_mesh
- added link inkcap_left_medium_0
- added link inkcap_left_small_0
- added link palette
- added link palette_mesh; visual mesh filename=meshes/palette/palette.obj scale=1 1 1
Joints:
- removed joint inkpalette_joint
- removed joint inkpalette_mesh_joint
- added joint inkcap_left_medium_0_joint: type fixed, parent palette, child inkcap_left_medium_0, origin xyz=-0.132 0.048 0 rpy=0 0 0
- added joint inkcap_left_small_0_joint: type fixed, parent palette, child inkcap_left_small_0, origin xyz=-0.15 0.037 0 rpy=0 0 0
- added joint palette_joint: type fixed, parent root, child palette, origin xyz=0 0 0 rpy=0 0 0
- added joint palette_mesh_joint: type fixed, parent palette, child palette_mesh, origin xyz=0 0 0 rpy=0 0 0
- joint inkcap_left_large_joint: origin xyz=-0.002 0.059 0 rpy=0 0 0 -> xyz=-0.15 0.025 0 rpy=0 0 0; parent inkpalette -> palette
- joint inkcap_left_medium_1_joint: origin xyz=-0.02 0.048 0 rpy=0 0 0 -> xyz=-0.15 0.048 0 rpy=0 0 0; parent inkpalette -> palette
- joint inkcap_left_medium_2_joint: origin xyz=-0.032 0.06 0 rpy=0 0 0 -> xyz=-0.168 0.048 0 rpy=0 0 0; parent inkpalette -> palette
- joint inkcap_left_small_1_joint: origin xyz=0.007 0.045 0 rpy=0 0 0 -> xyz=-0.15 0.049 0 rpy=0 0 0; parent inkpalette -> palette
- joint inkcap_left_small_2_joint: origin xyz=-0.012 0.074 0 rpy=0 0 0 -> xyz=-0.15 0.013 0 rpy=0 0 0; parent inkpalette -> palette
- joint inkcap_left_small_3_joint: origin xyz=-0.025 0.082 0 rpy=0 0 0 -> xyz=-0.15 0.001 0 rpy=0 0 0; parent inkpalette -> palette
- joint inkcap_right_large_joint: origin xyz=0.002 -0.059 0 rpy=0 0 0 -> xyz=-0.15 -0.025 0 rpy=0 0 0; parent inkpalette -> palette
- joint inkcap_right_medium_0_joint: origin xyz=0.02 -0.048 0 rpy=0 0 0 -> xyz=-0.132 -0.048 0 rpy=0 0 0; parent inkpalette -> palette
- joint inkcap_right_medium_1_joint: origin xyz=0.032 -0.06 0 rpy=0 0 0 -> xyz=-0.15 -0.048 0 rpy=0 0 0; parent inkpalette -> palette
- joint inkcap_right_medium_2_joint: origin xyz=0.015 -0.07 0 rpy=0 0 0 -> xyz=-0.168 -0.048 0 rpy=0 0 0; parent inkpalette -> palette
- joint inkcap_right_small_0_joint: origin xyz=-0.007 -0.045 0 rpy=0 0 0 -> xyz=-0.15 -0.013 0 rpy=0 0 0; parent inkpalette -> palette
- joint inkcap_right_small_1_joint: origin xyz=0.012 -0.074 0 rpy=0 0 0 -> xyz=-0.15 -0.001 0 rpy=0 0 0; parent inkpalette -> palette
- joint inkcap_right_small_2_joint: origin xyz=0.025 -0.082 0 rpy=0 0 0 -> xyz=-0.15 -0.037 0 rpy=0 0 0; parent inkpalette -> palette
- joint inkcap_right_small_3_joint: origin xyz=0.018 -0.065 0 rpy=0 0 0 -> xyz=-0.15 -0.049 0 rpy=0 0 0; parent inkpalette -> palette

Commit message: asd

File: urdf/tatbot.urdf (robot description, URDF)
Before this commit: robot tatbot, 92 links, 91 joints
Joints:
- joint inkcap_left_large_joint: origin xyz=-0.15 0.025 0 rpy=0 0 0 -> xyz=-0.13 0.025 0 rpy=0 0 0
- joint inkcap_left_medium_0_joint: origin xyz=-0.132 0.048 0 rpy=0 0 0 -> xyz=-0.112 0.048 0 rpy=0 0 0
- joint inkcap_left_medium_1_joint: origin xyz=-0.15 0.048 0 rpy=0 0 0 -> xyz=-0.13 0.048 0 rpy=0 0 0
- joint inkcap_left_medium_2_joint: origin xyz=-0.168 0.048 0 rpy=0 0 0 -> xyz=-0.148 0.048 0 rpy=0 0 0
- joint inkcap_left_small_0_joint: origin xyz=-0.15 0.037 0 rpy=0 0 0 -> xyz=-0.098 0.025 0 rpy=0 0 0
- joint inkcap_left_small_1_joint: origin xyz=-0.15 0.049 0 rpy=0 0 0 -> xyz=-0.118 0.025 0 rpy=0 0 0
- joint inkcap_left_small_2_joint: origin xyz=-0.15 0.013 0 rpy=0 0 0 -> xyz=-0.142 0.025 0 rpy=0 0 0
- joint inkcap_left_small_3_joint: origin xyz=-0.15 0.001 0 rpy=0 0 0 -> xyz=-0.162 0.025 0 rpy=0 0 0
- joint inkcap_right_large_joint: origin xyz=-0.15 -0.025 0 rpy=0 0 0 -> xyz=-0.13 -0.025 0 rpy=0 0 0
- joint inkcap_right_medium_0_joint: origin xyz=-0.132 -0.048 0 rpy=0 0 0 -> xyz=-0.112 -0.048 0 rpy=0 0 0
- joint inkcap_right_medium_1_joint: origin xyz=-0.15 -0.048 0 rpy=0 0 0 -> xyz=-0.13 -0.048 0 rpy=0 0 0
- joint inkcap_right_medium_2_joint: origin xyz=-0.168 -0.048 0 rpy=0 0 0 -> xyz=-0.148 -0.048 0 rpy=0 0 0
- joint inkcap_right_small_0_joint: origin xyz=-0.15 -0.013 0 rpy=0 0 0 -> xyz=-0.098 -0.025 0 rpy=0 0 0
- joint inkcap_right_small_1_joint: origin xyz=-0.15 -0.001 0 rpy=0 0 0 -> xyz=-0.118 -0.025 0 rpy=0 0 0
- joint inkcap_right_small_2_joint: origin xyz=-0.15 -0.037 0 rpy=0 0 0 -> xyz=-0.142 -0.025 0 rpy=0 0 0
- joint inkcap_right_small_3_joint: origin xyz=-0.15 -0.049 0 rpy=0 0 0 -> xyz=-0.162 -0.025 0 rpy=0 0 0

Commit message: taggy

File: urdf/tatbot.urdf (robot description, URDF)
Before this commit: robot tatbot, 92 links, 91 joints
Links:
- removed link palette_mesh
- link tag0: geometry visual mesh filename=meshes/tags/16h5_000_5cm/tag.obj scale=1 1 1
- link tag1: geometry visual mesh filename=meshes/tags/16h5_001_5cm/tag.obj scale=1 1 1
- link tag2: geometry visual mesh filename=meshes/tags/16h5_002_5cm/tag.obj scale=1 1 1
- link tag6: geometry visual mesh filename=meshes/tags/16h5_006_4cm/tag.obj scale=1 1 1
- link tag7: geometry visual mesh filename=meshes/tags/16h5_007_4cm/tag.obj scale=1 1 1
Joints:
- removed joint palette_mesh_joint
- joint tag0_joint: origin xyz=0 0 0.01 rpy=0 0 0 -> xyz=-0.04 0 0.01 rpy=0 0 0

Commit message: ink viz working

File: urdf/tatbot.urdf (robot description, URDF)
Before this commit: robot tatbot, 91 links, 90 joints
Links:
- added link palette_mesh; visual mesh filename=meshes/palette/palette.obj scale=1 1 1
Joints:
- added joint palette_mesh_joint: type fixed, parent palette, child palette_mesh, origin xyz=0 0 0 rpy=0 0 0

Commit message: asd

File: urdf/tatbot.urdf (robot description, URDF)
Before this commit: robot tatbot, 92 links, 91 joints
Joints:
- joint realsense1_joint: origin xyz=-0.22 0 0.2 rpy=0 0.7853981633974483 0 -> xyz=0.2 0.15 0.05 rpy=0 0.7853981633974483 -2.3

Commit message: Add retracted poses for left and right configurations, update default scene references, and modify URDF for new tags

File: urdf/tatbot.urdf (robot description, URDF)
Before this commit: robot tatbot, 92 links, 91 joints
Links:
- removed link palette_mesh
- added link tag3; visual mesh filename=meshes/tags/16h5_003_5cm/tag.obj scale=1 1 1
Joints:
- removed joint palette_mesh_joint
- added joint tag3_joint: type fixed, parent root, child tag3, origin xyz=0.06 0 0 rpy=0 0 0
- joint tag0_joint: origin xyz=-0.04 0 0.01 rpy=0 0 0 -> xyz=-0.02 0 0 rpy=0 0 0
- joint tag1_joint: origin xyz=0 0 0.01 rpy=0 0 0 -> xyz=0.02 0 0.025 rpy=0 -1.57 0
- joint tag2_joint: origin xyz=0 0 0.01 rpy=0 0 0 -> xyz=0.03 0 0.025 rpy=0 1.57 0

Commit message: asd

File: urdf/tatbot.urdf (robot description, URDF)
Before this commit: robot tatbot, 92 links, 91 joints
Joints:
- joint inkcap_left_large_joint: origin xyz=-0.13 0.025 0 rpy=0 0 0 -> xyz=-0.11 0.025 0 rpy=0 0 0
- joint inkcap_left_medium_0_joint: origin xyz=-0.112 0.048 0 rpy=0 0 0 -> xyz=-0.092 0.053 0 rpy=0 0 0
- joint inkcap_left_medium_1_joint: origin xyz=-0.13 0.048 0 rpy=0 0 0 -> xyz=-0.11 0.048 0 rpy=0 0 0
- joint inkcap_left_medium_2_joint: origin xyz=-0.148 0.048 0 rpy=0 0 0 -> xyz=-0.128 0.053 0 rpy=0 0 0
- joint inkcap_left_small_0_joint: origin xyz=-0.098 0.025 0 rpy=0 0 0 -> xyz=-0.078 0.035 0 rpy=0 0 0
- joint inkcap_left_small_1_joint: origin xyz=-0.118 0.025 0 rpy=0 0 0 -> xyz=-0.093 0.03 0 rpy=0 0 0
- joint inkcap_left_small_2_joint: origin xyz=-0.142 0.025 0 rpy=0 0 0 -> xyz=-0.127 0.03 0 rpy=0 0 0
- joint inkcap_left_small_3_joint: origin xyz=-0.162 0.025 0 rpy=0 0 0 -> xyz=-0.142 0.035 0 rpy=0 0 0
- joint inkcap_right_large_joint: origin xyz=-0.13 -0.025 0 rpy=0 0 0 -> xyz=-0.11 -0.025 0 rpy=0 0 0
- joint inkcap_right_medium_0_joint: origin xyz=-0.112 -0.048 0 rpy=0 0 0 -> xyz=-0.092 -0.053 0 rpy=0 0 0
- joint inkcap_right_medium_1_joint: origin xyz=-0.13 -0.048 0 rpy=0 0 0 -> xyz=-0.11 -0.048 0 rpy=0 0 0
- joint inkcap_right_medium_2_joint: origin xyz=-0.148 -0.048 0 rpy=0 0 0 -> xyz=-0.128 -0.053 0 rpy=0 0 0
- joint inkcap_right_small_0_joint: origin xyz=-0.098 -0.025 0 rpy=0 0 0 -> xyz=-0.078 -0.035 0 rpy=0 0 0
- joint inkcap_right_small_1_joint: origin xyz=-0.118 -0.025 0 rpy=0 0 0 -> xyz=-0.093 -0.03 0 rpy=0 0 0
- joint inkcap_right_small_2_joint: origin xyz=-0.142 -0.025 0 rpy=0 0 0 -> xyz=-0.127 -0.03 0 rpy=0 0 0
- joint inkcap_right_small_3_joint: origin xyz=-0.162 -0.025 0 rpy=0 0 0 -> xyz=-0.142 -0.035 0 rpy=0 0 0

Commit message: asd

File: urdf/tatbot.urdf (robot description, URDF)
Before this commit: robot tatbot, 92 links, 91 joints
Joints:
- joint inkcap_left_large_joint: origin xyz=-0.11 0.025 0 rpy=0 0 0 -> xyz=-0.11 0.025 0.005 rpy=0 0 0
- joint inkcap_left_medium_0_joint: origin xyz=-0.092 0.053 0 rpy=0 0 0 -> xyz=-0.092 0.053 0.005 rpy=0 0 0
- joint inkcap_left_medium_1_joint: origin xyz=-0.11 0.048 0 rpy=0 0 0 -> xyz=-0.11 0.048 0.005 rpy=0 0 0
- joint inkcap_left_medium_2_joint: origin xyz=-0.128 0.053 0 rpy=0 0 0 -> xyz=-0.128 0.053 0.005 rpy=0 0 0
- joint inkcap_left_small_0_joint: origin xyz=-0.078 0.035 0 rpy=0 0 0 -> xyz=-0.078 0.035 0.005 rpy=0 0 0
- joint inkcap_left_small_1_joint: origin xyz=-0.093 0.03 0 rpy=0 0 0 -> xyz=-0.093 0.03 0.005 rpy=0 0 0
- joint inkcap_left_small_2_joint: origin xyz=-0.127 0.03 0 rpy=0 0 0 -> xyz=-0.127 0.03 0.005 rpy=0 0 0
- joint inkcap_left_small_3_joint: origin xyz=-0.142 0.035 0 rpy=0 0 0 -> xyz=-0.142 0.035 0.005 rpy=0 0 0
- joint inkcap_right_large_joint: origin xyz=-0.11 -0.025 0 rpy=0 0 0 -> xyz=-0.11 -0.025 0.005 rpy=0 0 0
- joint inkcap_right_medium_0_joint: origin xyz=-0.092 -0.053 0 rpy=0 0 0 -> xyz=-0.092 -0.053 0.005 rpy=0 0 0
- joint inkcap_right_medium_1_joint: origin xyz=-0.11 -0.048 0 rpy=0 0 0 -> xyz=-0.11 -0.048 0.005 rpy=0 0 0
- joint inkcap_right_medium_2_joint: origin xyz=-0.128 -0.053 0 rpy=0 0 0 -> xyz=-0.128 -0.053 0.005 rpy=0 0 0
- joint inkcap_right_small_0_joint: origin xyz=-0.078 -0.035 0 rpy=0 0 0 -> xyz=-0.078 -0.035 0.005 rpy=0 0 0
- joint inkcap_right_small_1_joint: origin xyz=-0.093 -0.03 0 rpy=0 0 0 -> xyz=-0.093 -0.03 0.005 rpy=0 0 0
- joint inkcap_right_small_2_joint: origin xyz=-0.127 -0.03 0 rpy=0 0 0 -> xyz=-0.127 -0.03 0.005 rpy=0 0 0
- joint inkcap_right_small_3_joint: origin xyz=-0.142 -0.035 0 rpy=0 0 0 -> xyz=-0.142 -0.035 0.005 rpy=0 0 0

Commit message: asd

File: urdf/tatbot.urdf (robot description, URDF)
Before this commit: robot tatbot, 92 links, 91 joints
Joints:
- joint left/left_index_joint: axis 0 0 0 -> (none)
- joint left/right_carriage_joint: limit lower=0.0 upper=0.001 effort=400.0 velocity=0.0875 -> lower=0.0 upper=0.04 effort=400.0 velocity=0.0875
- joint right/left_carriage_joint: limit lower=0.0 upper=0.001 effort=400.0 velocity=0.0875 -> lower=0.0 upper=0.044 effort=400.0 velocity=0.0875
- joint right/right_carriage_joint: limit lower=0.0 upper=0.001 effort=400.0 velocity=0.0875 -> lower=0.0 upper=0.044 effort=400.0 velocity=0.0875
- joint right/right_index_joint: axis 0 0 0 -> (none)

Commit message: asd

File: urdf/tatbot.urdf (robot description, URDF)
Before this commit: robot tatbot, 92 links, 91 joints
Joints:
- joint inkcap_left_large_joint: origin xyz=-0.11 0.025 0.005 rpy=0 0 0 -> xyz=-0.11 0.025 0.009 rpy=0 0 0
- joint inkcap_left_medium_0_joint: origin xyz=-0.092 0.053 0.005 rpy=0 0 0 -> xyz=-0.092 0.053 0.009 rpy=0 0 0
- joint inkcap_left_medium_1_joint: origin xyz=-0.11 0.048 0.005 rpy=0 0 0 -> xyz=-0.11 0.048 0.009 rpy=0 0 0
- joint inkcap_left_medium_2_joint: origin xyz=-0.128 0.053 0.005 rpy=0 0 0 -> xyz=-0.128 0.053 0.009 rpy=0 0 0
- joint inkcap_left_small_0_joint: origin xyz=-0.078 0.035 0.005 rpy=0 0 0 -> xyz=-0.078 0.035 0.009 rpy=0 0 0
- joint inkcap_left_small_1_joint: origin xyz=-0.093 0.03 0.005 rpy=0 0 0 -> xyz=-0.093 0.03 0.009 rpy=0 0 0
- joint inkcap_left_small_2_joint: origin xyz=-0.127 0.03 0.005 rpy=0 0 0 -> xyz=-0.127 0.03 0.009 rpy=0 0 0
- joint inkcap_left_small_3_joint: origin xyz=-0.142 0.035 0.005 rpy=0 0 0 -> xyz=-0.142 0.035 0.009 rpy=0 0 0
- joint inkcap_right_large_joint: origin xyz=-0.11 -0.025 0.005 rpy=0 0 0 -> xyz=-0.11 -0.025 0.009 rpy=0 0 0
- joint inkcap_right_medium_0_joint: origin xyz=-0.092 -0.053 0.005 rpy=0 0 0 -> xyz=-0.092 -0.053 0.009 rpy=0 0 0
- joint inkcap_right_medium_1_joint: origin xyz=-0.11 -0.048 0.005 rpy=0 0 0 -> xyz=-0.11 -0.048 0.009 rpy=0 0 0
- joint inkcap_right_medium_2_joint: origin xyz=-0.128 -0.053 0.005 rpy=0 0 0 -> xyz=-0.128 -0.053 0.009 rpy=0 0 0
- joint inkcap_right_small_0_joint: origin xyz=-0.078 -0.035 0.005 rpy=0 0 0 -> xyz=-0.078 -0.035 0.009 rpy=0 0 0
- joint inkcap_right_small_1_joint: origin xyz=-0.093 -0.03 0.005 rpy=0 0 0 -> xyz=-0.093 -0.03 0.009 rpy=0 0 0
- joint inkcap_right_small_2_joint: origin xyz=-0.127 -0.03 0.005 rpy=0 0 0 -> xyz=-0.127 -0.03 0.009 rpy=0 0 0
- joint inkcap_right_small_3_joint: origin xyz=-0.142 -0.035 0.005 rpy=0 0 0 -> xyz=-0.142 -0.035 0.009 rpy=0 0 0

Commit message: update urdf

File: urdf/tatbot.urdf (robot description, URDF)
Before this commit: robot tatbot, 92 links, 91 joints
Links:
- removed link 300mm_left_rail_left
- removed link 300mm_left_rail_right
- removed link 300mm_right_rail_left
- removed link 300mm_right_rail_right
- removed link 300mm_vertical_top
- added link 300mm_front_rail_left; visual mesh filename=meshes/frame/t2020_300mm.stl scale=0.001 0.001 0.001
- added link 300mm_front_rail_right; visual mesh filename=meshes/frame/t2020_300mm.stl scale=0.001 0.001 0.001
- added link 600mm_vertical_top; visual mesh filename=meshes/frame/t2020_600mm.stl scale=0.001 0.001 0.001
Joints:
- removed joint 300mm_left_rail_left_joint
- removed joint 300mm_left_rail_right_joint
- removed joint 300mm_right_rail_left_joint
- removed joint 300mm_right_rail_right_joint
- removed joint 300mm_vertical_top_joint
- added joint 300mm_front_rail_left_joint: type fixed, parent root, child 300mm_front_rail_left, origin xyz=0.08 0.1 -0.01 rpy=0 0 0
- added joint 300mm_front_rail_right_joint: type fixed, parent root, child 300mm_front_rail_right, origin xyz=0.08 -0.1 -0.01 rpy=0 0 0
- added joint 600mm_vertical_top_joint: type fixed, parent root, child 600mm_vertical_top, origin xyz=-0.0275 0 0.61 rpy=0 0 0
- joint 600mm_back_horizontal_joint: origin xyz=-0.267 0 -0.03 rpy=0 0 0 -> xyz=-0.0275 0 -0.01 rpy=0 0 0
- joint 600mm_front_horizontal_joint: origin xyz=0.0278 0 -0.03 rpy=0 0 0 -> xyz=0.0275 0 -0.01 rpy=0 0 0
- joint 600mm_vertical_left_joint: origin xyz=-0.267 0.08128 0.28 rpy=0 0 0 -> xyz=-0.0275 0.1 0.30 rpy=0 0 0
- joint 600mm_vertical_right_joint: origin xyz=-0.267 -0.08128 0.28 rpy=0 0 0 -> xyz=-0.0275 -0.1 0.30 rpy=0 0 0
- joint camera1_mount_joint: origin xyz=0.0378 0.258125 -0.08 rpy=0 1.5707963267948966 0 -> xyz=-0.0275 0.09 0.2 rpy=0 1.5707963267948966 -1.5707963267948966
- joint camera2_mount_joint: origin xyz=-0.257 0.08128 0.5 rpy=0 1.5707963267948966 0 -> xyz=-0.0275 0.27 0.6 rpy=0 1.5707963267948966 0
- joint camera3_mount_joint: origin xyz=-0.257 0.06 0.7 rpy=0 1.5707963267948966 0 -> xyz=-0.0275 0.11 0.7 rpy=0 1.5707963267948966 0
- joint camera4_mount_joint: origin xyz=-0.257 -0.06 0.7 rpy=0 1.5707963267948966 0 -> xyz=-0.0275 -0.11 0.7 rpy=0 1.5707963267948966 0
- joint camera5_mount_joint: origin xyz=0.0378 -0.258125 -0.08 rpy=0 1.5707963267948966 0 -> xyz=-0.0275 -0.27 0.6 rpy=0 1.5707963267948966 0
- joint left/mount_joint: origin xyz=0 0.238125 0 rpy=0 0 0 -> xyz=0 0.2675 0 rpy=0 0 0
- joint right/mount_joint: origin xyz=0 -0.238125 0 rpy=0 0 0 -> xyz=0 -0.2675 0 rpy=0 0 0
