Commit message: mounted realsenses

File: urdf/tatbot.urdf (robot description, URDF)
Before this commit: robot tatbot, 90 links, 89 joints
Links:
- removed link realsense1_bottom_screw_frame
- removed link realsense1_color_frame
- removed link realsense1_color_optical_frame
- removed link realsense1_depth_frame
- removed link realsense1_depth_optical_frame
- removed link realsense1_infra1_frame
- removed link realsense1_infra1_optical_frame
- removed link realsense1_infra2_frame
- removed link realsense1_infra2_optical_frame
- removed link realsense1_link
- removed link realsense2_bottom_screw_frame
- removed link realsense2_color_frame
- removed link realsense2_color_optical_frame
- removed link realsense2_depth_frame
- removed link realsense2_depth_optical_frame
- removed link realsense2_infra1_frame
- removed link realsense2_infra1_optical_frame
- removed link realsense2_infra2_frame
- removed link realsense2_infra2_optical_frame
- removed link realsense2_link
- removed link tag6
- removed link tag7
- added link left/realsense_bottom_screw_frame
- added link left/realsense_color_frame
- added link left/realsense_color_optical_frame
- added link left/realsense_depth_frame
- added link left/realsense_depth_optical_frame
- added link left/realsense_infra1_frame
- added link left/realsense_infra1_optical_frame
- added link left/realsense_infra2_frame
- added link left/realsense_infra2_optical_frame
- added link left/realsense_link, mass 0.072; collision box size=0.023 0.042 0.042; visual mesh filename=meshes/cameras/d405.stl scale=0.001 0.001 0.001
- added link left/realsense_mount_d405, mass 0.04518012; collision mesh filename=meshes/wxai/camera_mount_d405.stl; visual mesh filename=meshes/wxai/camera_mount_d405.stl
- added link right/realsense_bottom_screw_frame
- added link right/realsense_color_frame
- added link right/realsense_color_optical_frame
- added link right/realsense_depth_frame
- added link right/realsense_depth_optical_frame
- added link right/realsense_infra1_frame
- added link right/realsense_infra1_optical_frame
- added link right/realsense_infra2_frame
- added link right/realsense_infra2_optical_frame
- added link right/realsense_link, mass 0.072; collision box size=0.023 0.042 0.042; visual mesh filename=meshes/cameras/d405.stl scale=0.001 0.001 0.001
- added link right/realsense_mount_d405, mass 0.04518012; collision mesh filename=meshes/wxai/camera_mount_d405.stl; visual mesh filename=meshes/wxai/camera_mount_d405.stl
Joints:
- removed joint realsense1_color_joint
- removed joint realsense1_color_optical_joint
- removed joint realsense1_depth_joint
- removed joint realsense1_depth_optical_joint
- removed joint realsense1_infra1_joint
- removed joint realsense1_infra1_optical_joint
- removed joint realsense1_infra2_joint
- removed joint realsense1_infra2_optical_joint
- removed joint realsense1_joint
- removed joint realsense1_link_joint
- removed joint realsense2_color_joint
- removed joint realsense2_color_optical_joint
- removed joint realsense2_depth_joint
- removed joint realsense2_depth_optical_joint
- removed joint realsense2_infra1_joint
- removed joint realsense2_infra1_optical_joint
- removed joint realsense2_infra2_joint
- removed joint realsense2_infra2_optical_joint
- removed joint realsense2_joint
- removed joint realsense2_link_joint
- removed joint tag6_joint
- removed joint tag7_joint
- added joint left/realsense_color_joint: type fixed, parent left/realsense_link, child left/realsense_color_frame, origin xyz=0 0.0 0 rpy=0 0 0
- added joint left/realsense_color_optical_joint: type fixed, parent left/realsense_color_frame, child left/realsense_color_optical_frame, origin xyz=0 0 0 rpy=-1.5707963267948966 0 -1.5707963267948966
- added joint left/realsense_depth_joint: type fixed, parent left/realsense_link, child left/realsense_depth_frame, origin xyz=0 0 0 rpy=0 0 0
- added joint left/realsense_depth_optical_joint: type fixed, parent left/realsense_depth_frame, child left/realsense_depth_optical_frame, origin xyz=0 0 0 rpy=-1.5707963267948966 0 -1.5707963267948966
- added joint left/realsense_infra1_joint: type fixed, parent left/realsense_link, child left/realsense_infra1_frame, origin xyz=0 0.0 0 rpy=0 0 0
- added joint left/realsense_infra1_optical_joint: type fixed, parent left/realsense_infra1_frame, child left/realsense_infra1_optical_frame, origin xyz=0 0 0 rpy=-1.5707963267948966 0 -1.5707963267948966
- added joint left/realsense_infra2_joint: type fixed, parent left/realsense_link, child left/realsense_infra2_frame, origin xyz=0 -0.018 0 rpy=0 0 0
- added joint left/realsense_infra2_optical_joint: type fixed, parent left/realsense_infra2_frame, child left/realsense_infra2_optical_frame, origin xyz=0 0 0 rpy=-1.5707963267948966 0 -1.5707963267948966
- added joint left/realsense_joint: type fixed, parent left/realsense_mount_d405, child left/realsense_bottom_screw_frame, origin xyz=0.02927207801 0 0.03824951197 rpy=0 0.3490658503988659 0
- added joint left/realsense_link_joint: type fixed, parent left/realsense_bottom_screw_frame, child left/realsense_link, origin xyz=0.01085 0.009 0.021 rpy=0 0 0
- added joint left/realsense_mount_joint: type fixed, parent left/link_6, child left/realsense_mount_d405, origin xyz=0.012 0 0 rpy=0 0 0
- added joint right/realsense_color_joint: type fixed, parent right/realsense_link, child right/realsense_color_frame, origin xyz=0 0.0 0 rpy=0 0 0
- added joint right/realsense_color_optical_joint: type fixed, parent right/realsense_color_frame, child right/realsense_color_optical_frame, origin xyz=0 0 0 rpy=-1.5707963267948966 0 -1.5707963267948966
- added joint right/realsense_depth_joint: type fixed, parent right/realsense_link, child right/realsense_depth_frame, origin xyz=0 0 0 rpy=0 0 0
- added joint right/realsense_depth_optical_joint: type fixed, parent right/realsense_depth_frame, child right/realsense_depth_optical_frame, origin xyz=0 0 0 rpy=-1.5707963267948966 0 -1.5707963267948966
- added joint right/realsense_infra1_joint: type fixed, parent right/realsense_link, child right/realsense_infra1_frame, origin xyz=0 0.0 0 rpy=0 0 0
- added joint right/realsense_infra1_optical_joint: type fixed, parent right/realsense_infra1_frame, child right/realsense_infra1_optical_frame, origin xyz=0 0 0 rpy=-1.5707963267948966 0 -1.5707963267948966
- added joint right/realsense_infra2_joint: type fixed, parent right/realsense_link, child right/realsense_infra2_frame, origin xyz=0 -0.018 0 rpy=0 0 0
- added joint right/realsense_infra2_optical_joint: type fixed, parent right/realsense_infra2_frame, child right/realsense_infra2_optical_frame, origin xyz=0 0 0 rpy=-1.5707963267948966 0 -1.5707963267948966
- added joint right/realsense_joint: type fixed, parent right/realsense_mount_d405, child right/realsense_bottom_screw_frame, origin xyz=0.02927207801 0 0.03824951197 rpy=0 0.3490658503988659 0
- added joint right/realsense_link_joint: type fixed, parent right/realsense_bottom_screw_frame, child right/realsense_link, origin xyz=0.01085 0.009 0.021 rpy=0 0 0
- added joint right/realsense_mount_joint: type fixed, parent right/link_6, child right/realsense_mount_d405, origin xyz=0.012 0 0 rpy=0 0 0

Commit message: asd

File: urdf/tatbot.urdf (robot description, URDF)
Before this commit: robot tatbot, 90 links, 89 joints
Links:
- link left/leader_finger_left_thumb: geometry collision mesh filename=meshes/wxai/leader_finger_left_thumb.stl
- link left/tattoo_needle: geometry collision cylinder length=0.035 radius=0.002
- link left/tattoo_pen: geometry collision cylinder length=0.1 radius=0.012
- link right/leader_finger_right_thumb: geometry collision mesh filename=meshes/wxai/leader_finger_right_thumb.stl
- link right/tattoo_needle: geometry collision cylinder length=0.035 radius=0.002
- link right/tattoo_pen: geometry collision cylinder length=0.1 radius=0.012

Commit message: asd

File: urdf/tatbot.urdf (robot description, URDF)
Before this commit: robot tatbot, 90 links, 89 joints
Links:
- removed link inkcap_left_medium_2
- removed link inkcap_right_medium_2
Joints:
- removed joint inkcap_left_medium_2_joint
- removed joint inkcap_right_medium_2_joint
- joint inkcap_left_large_joint: origin xyz=-0.11 0.025 0.009 rpy=0 0 0 -> xyz=0.08 0.051 0.054 rpy=0 0 0
- joint inkcap_left_medium_0_joint: origin xyz=-0.092 0.053 0.009 rpy=0 0 0 -> xyz=0.06 0.051 0.054 rpy=0 0 0
- joint inkcap_left_medium_1_joint: origin xyz=-0.11 0.048 0.009 rpy=0 0 0 -> xyz=0.1 0.051 0.054 rpy=0 0 0
- joint inkcap_left_small_0_joint: origin xyz=-0.078 0.035 0.009 rpy=0 0 0 -> xyz=0.056 0.027 0.054 rpy=0 0 0
- joint inkcap_left_small_1_joint: origin xyz=-0.093 0.03 0.009 rpy=0 0 0 -> xyz=0.072 0.027 0.054 rpy=0 0 0
- joint inkcap_left_small_2_joint: origin xyz=-0.127 0.03 0.009 rpy=0 0 0 -> xyz=0.088 0.027 0.054 rpy=0 0 0
- joint inkcap_left_small_3_joint: origin xyz=-0.142 0.035 0.009 rpy=0 0 0 -> xyz=0.104 0.027 0.054 rpy=0 0 0
- joint inkcap_right_large_joint: origin xyz=-0.11 -0.025 0.009 rpy=0 0 0 -> xyz=0.08 -0.051 0.054 rpy=0 0 0
- joint inkcap_right_medium_0_joint: origin xyz=-0.092 -0.053 0.009 rpy=0 0 0 -> xyz=0.06 -0.051 0.054 rpy=0 0 0
- joint inkcap_right_medium_1_joint: origin xyz=-0.11 -0.048 0.009 rpy=0 0 0 -> xyz=0.1 -0.051 0.054 rpy=0 0 0
- joint inkcap_right_small_0_joint: origin xyz=-0.078 -0.035 0.009 rpy=0 0 0 -> xyz=0.056 -0.027 0.054 rpy=0 0 0
- joint inkcap_right_small_1_joint: origin xyz=-0.093 -0.03 0.009 rpy=0 0 0 -> xyz=0.072 -0.027 0.054 rpy=0 0 0
- joint inkcap_right_small_2_joint: origin xyz=-0.127 -0.03 0.009 rpy=0 0 0 -> xyz=0.088 -0.027 0.054 rpy=0 0 0
- joint inkcap_right_small_3_joint: origin xyz=-0.142 -0.035 0.009 rpy=0 0 0 -> xyz=0.104 -0.027 0.054 rpy=0 0 0

Commit message: new ee

File: urdf/tatbot.urdf (robot description, URDF)
Before this commit: robot tatbot, 88 links, 87 joints
Links:
- removed link left/carriage_right
- removed link left/leader_finger_left_thumb
- removed link right/carriage_left
- removed link right/leader_finger_right_thumb
- added link left/ee_p1; visual mesh filename=meshes/ee/p1.stl scale=0.001 0.001 0.001
- added link left/ee_p2; visual mesh filename=meshes/ee/p2.stl scale=0.001 0.001 0.001
- added link right/ee_p1; visual mesh filename=meshes/ee/p1.stl scale=0.001 0.001 0.001
- added link right/ee_p2; visual mesh filename=meshes/ee/p2.stl scale=0.001 0.001 0.001
- link left/tattoo_needle: geometry visual cylinder length=0.035 radius=0.002
- link left/tattoo_pen: mass 0.01 -> None; geometry visual cylinder length=0.08 radius=0.015
- link right/tattoo_needle: geometry visual cylinder length=0.035 radius=0.002
- link right/tattoo_pen: mass 0.01 -> None; geometry visual cylinder length=0.08 radius=0.015
Joints:
- removed joint left/left_index_joint
- removed joint left/right_carriage_joint
- removed joint right/left_carriage_joint
- removed joint right/right_index_joint
- added joint left/ee_p1_joint: type fixed, parent left/carriage_left, child left/ee_p1, origin xyz=0 0 0 rpy=0 0 0
- added joint left/ee_p2_joint: type fixed, parent left/ee_p1, child left/ee_p2, origin xyz=0 0 0 rpy=0 0 0
- added joint right/ee_p1_joint: type fixed, parent right/carriage_right, child right/ee_p1, origin xyz=0 0 0 rpy=0 0 0
- added joint right/ee_p2_joint: type fixed, parent right/ee_p1, child right/ee_p2, origin xyz=0 0 0 rpy=0 0 0
- joint left/left_carriage_joint: limit lower=0.0 upper=0.001 effort=400.0 velocity=0.0875 -> lower=0.0 upper=0.044 effort=400.0 velocity=0.0875
- joint left/tattoo_needle_joint: origin xyz=0.035 0 0 rpy=0 0 0 -> xyz=0 0 -0.057 rpy=0 0 0
- joint left/tattoo_pen_joint: origin xyz=0.1 -0.01 0.055 rpy=0 0 0 -> xyz=0.061 0.041 0 rpy=-1.5707963267948966 0 0.7853981633974483; parent left/leader_finger_left_thumb -> left/ee_p1
- joint right/tattoo_needle_joint: origin xyz=0.035 0 0 rpy=0 0 0 -> xyz=0 0 -0.057 rpy=0 0 0
- joint right/tattoo_pen_joint: origin xyz=0.1 0.01 0.055 rpy=0 0 0 -> xyz=0.061 -0.041 0 rpy=1.5707963267948966 0 -0.7853981633974483; parent right/leader_finger_right_thumb -> right/ee_p1

Commit message: asd

File: urdf/tatbot.urdf (robot description, URDF)
Before this commit: robot tatbot, 88 links, 87 joints
Joints:
- joint left/tattoo_needle_joint: origin xyz=0 0 -0.057 rpy=0 0 0 -> xyz=0 0 -0.065 rpy=0 0 0
- joint left/tattoo_pen_joint: origin xyz=0.061 0.041 0 rpy=-1.5707963267948966 0 0.7853981633974483 -> xyz=0.051 0.051 0 rpy=-1.5707963267948966 0 0.7853981633974483
- joint right/tattoo_needle_joint: origin xyz=0 0 -0.057 rpy=0 0 0 -> xyz=0 0 -0.065 rpy=0 0 0
- joint right/tattoo_pen_joint: origin xyz=0.061 -0.041 0 rpy=1.5707963267948966 0 -0.7853981633974483 -> xyz=0.051 -0.051 0 rpy=1.5707963267948966 0 -0.7853981633974483

Commit message: better camera frustrums

File: urdf/tatbot.urdf (robot description, URDF)
Before this commit: robot tatbot, 88 links, 87 joints
Joints:
- joint camera1_frame_joint: origin xyz=0 0 0 rpy=0 0 0 -> xyz=0 0 0.07 rpy=-1.5707963267948966 0 0.7853981633974483
- joint camera2_frame_joint: origin xyz=0 0 0 rpy=0 0 0 -> xyz=0 0 0.07 rpy=0 0 0
- joint camera3_frame_joint: origin xyz=0 0 0 rpy=0 0 0 -> xyz=0 0 0.07 rpy=0 0 0
- joint camera4_frame_joint: origin xyz=0 0 0 rpy=0 0 0 -> xyz=0 0 0.07 rpy=0 0 0
- joint camera5_frame_joint: origin xyz=0 0 0 rpy=0 0 0 -> xyz=0 0 0.07 rpy=0 0 0

Commit message: asd

File: urdf/tatbot.urdf (robot description, URDF)
Before this commit: robot tatbot, 88 links, 87 joints
Joints:
- joint inkcap_left_large_joint: origin xyz=0.08 0.051 0.054 rpy=0 0 0 -> xyz=0.08 0.051 0.08 rpy=0 0 0
- joint inkcap_left_medium_0_joint: origin xyz=0.06 0.051 0.054 rpy=0 0 0 -> xyz=0.06 0.051 0.08 rpy=0 0 0
- joint inkcap_left_medium_1_joint: origin xyz=0.1 0.051 0.054 rpy=0 0 0 -> xyz=0.1 0.051 0.08 rpy=0 0 0
- joint inkcap_left_small_0_joint: origin xyz=0.056 0.027 0.054 rpy=0 0 0 -> xyz=0.056 0.027 0.08 rpy=0 0 0
- joint inkcap_left_small_1_joint: origin xyz=0.072 0.027 0.054 rpy=0 0 0 -> xyz=0.072 0.027 0.08 rpy=0 0 0
- joint inkcap_left_small_2_joint: origin xyz=0.088 0.027 0.054 rpy=0 0 0 -> xyz=0.088 0.027 0.08 rpy=0 0 0
- joint inkcap_left_small_3_joint: origin xyz=0.104 0.027 0.054 rpy=0 0 0 -> xyz=0.104 0.027 0.08 rpy=0 0 0
- joint inkcap_right_large_joint: origin xyz=0.08 -0.051 0.054 rpy=0 0 0 -> xyz=0.08 -0.051 0.08 rpy=0 0 0
- joint inkcap_right_medium_0_joint: origin xyz=0.06 -0.051 0.054 rpy=0 0 0 -> xyz=0.06 -0.051 0.08 rpy=0 0 0
- joint inkcap_right_medium_1_joint: origin xyz=0.1 -0.051 0.054 rpy=0 0 0 -> xyz=0.1 -0.051 0.08 rpy=0 0 0
- joint inkcap_right_small_0_joint: origin xyz=0.056 -0.027 0.054 rpy=0 0 0 -> xyz=0.056 -0.027 0.08 rpy=0 0 0
- joint inkcap_right_small_1_joint: origin xyz=0.072 -0.027 0.054 rpy=0 0 0 -> xyz=0.072 -0.027 0.08 rpy=0 0 0
- joint inkcap_right_small_2_joint: origin xyz=0.088 -0.027 0.054 rpy=0 0 0 -> xyz=0.088 -0.027 0.08 rpy=0 0 0
- joint inkcap_right_small_3_joint: origin xyz=0.104 -0.027 0.054 rpy=0 0 0 -> xyz=0.104 -0.027 0.08 rpy=0 0 0

Commit message: asd

File: urdf/tatbot.urdf (robot description, URDF)
Before this commit: robot tatbot, 88 links, 87 joints
Joints:
- joint inkcap_left_large_joint: origin xyz=0.08 0.051 0.08 rpy=0 0 0 -> xyz=0.08 0.051 0.09 rpy=0 0 0
- joint inkcap_left_medium_0_joint: origin xyz=0.06 0.051 0.08 rpy=0 0 0 -> xyz=0.06 0.051 0.09 rpy=0 0 0
- joint inkcap_left_medium_1_joint: origin xyz=0.1 0.051 0.08 rpy=0 0 0 -> xyz=0.1 0.051 0.09 rpy=0 0 0
- joint inkcap_left_small_0_joint: origin xyz=0.056 0.027 0.08 rpy=0 0 0 -> xyz=0.056 0.027 0.09 rpy=0 0 0
- joint inkcap_left_small_1_joint: origin xyz=0.072 0.027 0.08 rpy=0 0 0 -> xyz=0.072 0.027 0.09 rpy=0 0 0
- joint inkcap_left_small_2_joint: origin xyz=0.088 0.027 0.08 rpy=0 0 0 -> xyz=0.088 0.027 0.09 rpy=0 0 0
- joint inkcap_left_small_3_joint: origin xyz=0.104 0.027 0.08 rpy=0 0 0 -> xyz=0.104 0.027 0.09 rpy=0 0 0
- joint inkcap_right_large_joint: origin xyz=0.08 -0.051 0.08 rpy=0 0 0 -> xyz=0.08 -0.051 0.09 rpy=0 0 0
- joint inkcap_right_medium_0_joint: origin xyz=0.06 -0.051 0.08 rpy=0 0 0 -> xyz=0.06 -0.051 0.09 rpy=0 0 0
- joint inkcap_right_medium_1_joint: origin xyz=0.1 -0.051 0.08 rpy=0 0 0 -> xyz=0.1 -0.051 0.09 rpy=0 0 0
- joint inkcap_right_small_0_joint: origin xyz=0.056 -0.027 0.08 rpy=0 0 0 -> xyz=0.056 -0.027 0.09 rpy=0 0 0
- joint inkcap_right_small_1_joint: origin xyz=0.072 -0.027 0.08 rpy=0 0 0 -> xyz=0.072 -0.027 0.09 rpy=0 0 0
- joint inkcap_right_small_2_joint: origin xyz=0.088 -0.027 0.08 rpy=0 0 0 -> xyz=0.088 -0.027 0.09 rpy=0 0 0
- joint inkcap_right_small_3_joint: origin xyz=0.104 -0.027 0.08 rpy=0 0 0 -> xyz=0.104 -0.027 0.09 rpy=0 0 0

Commit message: asd

File: urdf/tatbot.urdf (robot description, URDF)
Before this commit: robot tatbot, 88 links, 87 joints
Joints:
- joint inkcap_left_large_joint: origin xyz=0.08 0.051 0.09 rpy=0 0 0 -> xyz=0.09 0.051 0.09 rpy=0 0 0
- joint inkcap_left_medium_0_joint: origin xyz=0.06 0.051 0.09 rpy=0 0 0 -> xyz=0.07 0.051 0.09 rpy=0 0 0
- joint inkcap_left_medium_1_joint: origin xyz=0.1 0.051 0.09 rpy=0 0 0 -> xyz=0.11 0.051 0.09 rpy=0 0 0
- joint inkcap_left_small_0_joint: origin xyz=0.056 0.027 0.09 rpy=0 0 0 -> xyz=0.066 0.027 0.09 rpy=0 0 0
- joint inkcap_left_small_1_joint: origin xyz=0.072 0.027 0.09 rpy=0 0 0 -> xyz=0.082 0.027 0.09 rpy=0 0 0
- joint inkcap_left_small_2_joint: origin xyz=0.088 0.027 0.09 rpy=0 0 0 -> xyz=0.098 0.027 0.09 rpy=0 0 0
- joint inkcap_left_small_3_joint: origin xyz=0.104 0.027 0.09 rpy=0 0 0 -> xyz=0.114 0.027 0.09 rpy=0 0 0
- joint inkcap_right_large_joint: origin xyz=0.08 -0.051 0.09 rpy=0 0 0 -> xyz=0.09 -0.051 0.09 rpy=0 0 0
- joint inkcap_right_medium_0_joint: origin xyz=0.06 -0.051 0.09 rpy=0 0 0 -> xyz=0.07 -0.051 0.09 rpy=0 0 0
- joint inkcap_right_medium_1_joint: origin xyz=0.1 -0.051 0.09 rpy=0 0 0 -> xyz=0.11 -0.051 0.09 rpy=0 0 0
- joint inkcap_right_small_0_joint: origin xyz=0.056 -0.027 0.09 rpy=0 0 0 -> xyz=0.066 -0.027 0.09 rpy=0 0 0
- joint inkcap_right_small_1_joint: origin xyz=0.072 -0.027 0.09 rpy=0 0 0 -> xyz=0.082 -0.027 0.09 rpy=0 0 0
- joint inkcap_right_small_2_joint: origin xyz=0.088 -0.027 0.09 rpy=0 0 0 -> xyz=0.098 -0.027 0.09 rpy=0 0 0
- joint inkcap_right_small_3_joint: origin xyz=0.104 -0.027 0.09 rpy=0 0 0 -> xyz=0.114 -0.027 0.09 rpy=0 0 0

Commit message: asd

File: urdf/tatbot.urdf (robot description, URDF)
Before this commit: robot tatbot, 88 links, 87 joints
Joints:
- joint inkcap_left_large_joint: origin xyz=0.09 0.051 0.09 rpy=0 0 0 -> xyz=0.095 0.051 0.09 rpy=0 0 0
- joint inkcap_left_medium_0_joint: origin xyz=0.07 0.051 0.09 rpy=0 0 0 -> xyz=0.075 0.051 0.09 rpy=0 0 0
- joint inkcap_left_medium_1_joint: origin xyz=0.11 0.051 0.09 rpy=0 0 0 -> xyz=0.115 0.051 0.09 rpy=0 0 0
- joint inkcap_left_small_0_joint: origin xyz=0.066 0.027 0.09 rpy=0 0 0 -> xyz=0.071 0.027 0.09 rpy=0 0 0
- joint inkcap_left_small_1_joint: origin xyz=0.082 0.027 0.09 rpy=0 0 0 -> xyz=0.087 0.027 0.09 rpy=0 0 0
- joint inkcap_left_small_2_joint: origin xyz=0.098 0.027 0.09 rpy=0 0 0 -> xyz=0.103 0.027 0.09 rpy=0 0 0
- joint inkcap_left_small_3_joint: origin xyz=0.114 0.027 0.09 rpy=0 0 0 -> xyz=0.119 0.027 0.09 rpy=0 0 0
- joint inkcap_right_large_joint: origin xyz=0.09 -0.051 0.09 rpy=0 0 0 -> xyz=0.095 -0.051 0.09 rpy=0 0 0
- joint inkcap_right_medium_0_joint: origin xyz=0.07 -0.051 0.09 rpy=0 0 0 -> xyz=0.075 -0.051 0.09 rpy=0 0 0
- joint inkcap_right_medium_1_joint: origin xyz=0.11 -0.051 0.09 rpy=0 0 0 -> xyz=0.115 -0.051 0.09 rpy=0 0 0
- joint inkcap_right_small_0_joint: origin xyz=0.066 -0.027 0.09 rpy=0 0 0 -> xyz=0.071 -0.027 0.09 rpy=0 0 0
- joint inkcap_right_small_1_joint: origin xyz=0.082 -0.027 0.09 rpy=0 0 0 -> xyz=0.087 -0.027 0.09 rpy=0 0 0
- joint inkcap_right_small_2_joint: origin xyz=0.098 -0.027 0.09 rpy=0 0 0 -> xyz=0.103 -0.027 0.09 rpy=0 0 0
- joint inkcap_right_small_3_joint: origin xyz=0.114 -0.027 0.09 rpy=0 0 0 -> xyz=0.119 -0.027 0.09 rpy=0 0 0

Commit message: asd

File: urdf/tatbot.urdf (robot description, URDF)
Before this commit: robot tatbot, 88 links, 87 joints
Joints:
- joint inkcap_left_large_joint: origin xyz=0.095 0.051 0.09 rpy=0 0 0 -> xyz=0.095 0.048 0.09 rpy=0 0 0
- joint inkcap_left_medium_0_joint: origin xyz=0.075 0.051 0.09 rpy=0 0 0 -> xyz=0.075 0.048 0.09 rpy=0 0 0
- joint inkcap_left_medium_1_joint: origin xyz=0.115 0.051 0.09 rpy=0 0 0 -> xyz=0.115 0.048 0.09 rpy=0 0 0
- joint inkcap_right_large_joint: origin xyz=0.095 -0.051 0.09 rpy=0 0 0 -> xyz=0.095 -0.048 0.09 rpy=0 0 0
- joint inkcap_right_medium_0_joint: origin xyz=0.075 -0.051 0.09 rpy=0 0 0 -> xyz=0.075 -0.048 0.09 rpy=0 0 0
- joint inkcap_right_medium_1_joint: origin xyz=0.115 -0.051 0.09 rpy=0 0 0 -> xyz=0.115 -0.048 0.09 rpy=0 0 0

Commit message: asd

File: urdf/tatbot.urdf (robot description, URDF)
Before this commit: robot tatbot, 88 links, 87 joints
Joints:
- joint inkcap_left_large_joint: origin xyz=0.095 0.048 0.09 rpy=0 0 0 -> xyz=0.095 0.046 0.09 rpy=0 0 0
- joint inkcap_left_medium_0_joint: origin xyz=0.075 0.048 0.09 rpy=0 0 0 -> xyz=0.075 0.046 0.09 rpy=0 0 0
- joint inkcap_left_medium_1_joint: origin xyz=0.115 0.048 0.09 rpy=0 0 0 -> xyz=0.115 0.046 0.09 rpy=0 0 0
- joint inkcap_left_small_0_joint: origin xyz=0.071 0.027 0.09 rpy=0 0 0 -> xyz=0.071 0.025 0.09 rpy=0 0 0
- joint inkcap_left_small_1_joint: origin xyz=0.087 0.027 0.09 rpy=0 0 0 -> xyz=0.087 0.025 0.09 rpy=0 0 0
- joint inkcap_left_small_2_joint: origin xyz=0.103 0.027 0.09 rpy=0 0 0 -> xyz=0.103 0.025 0.09 rpy=0 0 0
- joint inkcap_left_small_3_joint: origin xyz=0.119 0.027 0.09 rpy=0 0 0 -> xyz=0.119 0.025 0.09 rpy=0 0 0
- joint inkcap_right_large_joint: origin xyz=0.095 -0.048 0.09 rpy=0 0 0 -> xyz=0.095 -0.046 0.09 rpy=0 0 0
- joint inkcap_right_medium_0_joint: origin xyz=0.075 -0.048 0.09 rpy=0 0 0 -> xyz=0.075 -0.046 0.09 rpy=0 0 0
- joint inkcap_right_medium_1_joint: origin xyz=0.115 -0.048 0.09 rpy=0 0 0 -> xyz=0.115 -0.046 0.09 rpy=0 0 0
- joint inkcap_right_small_0_joint: origin xyz=0.071 -0.027 0.09 rpy=0 0 0 -> xyz=0.071 -0.025 0.09 rpy=0 0 0
- joint inkcap_right_small_1_joint: origin xyz=0.087 -0.027 0.09 rpy=0 0 0 -> xyz=0.087 -0.025 0.09 rpy=0 0 0
- joint inkcap_right_small_2_joint: origin xyz=0.103 -0.027 0.09 rpy=0 0 0 -> xyz=0.103 -0.025 0.09 rpy=0 0 0
- joint inkcap_right_small_3_joint: origin xyz=0.119 -0.027 0.09 rpy=0 0 0 -> xyz=0.119 -0.025 0.09 rpy=0 0 0
