Commit message: asd

File: urdf/tatbot.urdf (robot description, URDF)
Before this commit: robot tatbot, 88 links, 87 joints
Joints:
- joint inkcap_left_large_joint: origin xyz=0.095 0.046 0.09 rpy=0 0 0 -> xyz=0.097 0.046 0.088 rpy=0 0 0
- joint inkcap_left_medium_0_joint: origin xyz=0.075 0.046 0.09 rpy=0 0 0 -> xyz=0.077 0.046 0.088 rpy=0 0 0
- joint inkcap_left_medium_1_joint: origin xyz=0.115 0.046 0.09 rpy=0 0 0 -> xyz=0.117 0.046 0.088 rpy=0 0 0
- joint inkcap_left_small_0_joint: origin xyz=0.071 0.025 0.09 rpy=0 0 0 -> xyz=0.073 0.025 0.088 rpy=0 0 0
- joint inkcap_left_small_1_joint: origin xyz=0.087 0.025 0.09 rpy=0 0 0 -> xyz=0.089 0.025 0.088 rpy=0 0 0
- joint inkcap_left_small_2_joint: origin xyz=0.103 0.025 0.09 rpy=0 0 0 -> xyz=0.105 0.025 0.088 rpy=0 0 0
- joint inkcap_left_small_3_joint: origin xyz=0.119 0.025 0.09 rpy=0 0 0 -> xyz=0.121 0.025 0.088 rpy=0 0 0
- joint inkcap_right_large_joint: origin xyz=0.095 -0.046 0.09 rpy=0 0 0 -> xyz=0.097 -0.046 0.088 rpy=0 0 0
- joint inkcap_right_medium_0_joint: origin xyz=0.075 -0.046 0.09 rpy=0 0 0 -> xyz=0.077 -0.046 0.088 rpy=0 0 0
- joint inkcap_right_medium_1_joint: origin xyz=0.115 -0.046 0.09 rpy=0 0 0 -> xyz=0.117 -0.046 0.088 rpy=0 0 0
- joint inkcap_right_small_0_joint: origin xyz=0.071 -0.025 0.09 rpy=0 0 0 -> xyz=0.073 -0.025 0.088 rpy=0 0 0
- joint inkcap_right_small_1_joint: origin xyz=0.087 -0.025 0.09 rpy=0 0 0 -> xyz=0.089 -0.025 0.088 rpy=0 0 0
- joint inkcap_right_small_2_joint: origin xyz=0.103 -0.025 0.09 rpy=0 0 0 -> xyz=0.105 -0.025 0.088 rpy=0 0 0
- joint inkcap_right_small_3_joint: origin xyz=0.119 -0.025 0.09 rpy=0 0 0 -> xyz=0.121 -0.025 0.088 rpy=0 0 0

Commit message: asd

File: urdf/tatbot.urdf (robot description, URDF)
Before this commit: robot tatbot, 88 links, 87 joints
Joints:
- joint inkcap_left_large_joint: origin xyz=0.097 0.046 0.088 rpy=0 0 0 -> xyz=0.099 0.046 0.088 rpy=0 0 0
- joint inkcap_left_medium_0_joint: origin xyz=0.077 0.046 0.088 rpy=0 0 0 -> xyz=0.079 0.046 0.088 rpy=0 0 0
- joint inkcap_left_medium_1_joint: origin xyz=0.117 0.046 0.088 rpy=0 0 0 -> xyz=0.119 0.046 0.088 rpy=0 0 0
- joint inkcap_left_small_0_joint: origin xyz=0.073 0.025 0.088 rpy=0 0 0 -> xyz=0.075 0.025 0.088 rpy=0 0 0
- joint inkcap_left_small_1_joint: origin xyz=0.089 0.025 0.088 rpy=0 0 0 -> xyz=0.091 0.025 0.088 rpy=0 0 0
- joint inkcap_left_small_2_joint: origin xyz=0.105 0.025 0.088 rpy=0 0 0 -> xyz=0.107 0.025 0.088 rpy=0 0 0
- joint inkcap_left_small_3_joint: origin xyz=0.121 0.025 0.088 rpy=0 0 0 -> xyz=0.123 0.025 0.088 rpy=0 0 0
- joint inkcap_right_large_joint: origin xyz=0.097 -0.046 0.088 rpy=0 0 0 -> xyz=0.099 -0.046 0.088 rpy=0 0 0
- joint inkcap_right_medium_0_joint: origin xyz=0.077 -0.046 0.088 rpy=0 0 0 -> xyz=0.079 -0.046 0.088 rpy=0 0 0
- joint inkcap_right_medium_1_joint: origin xyz=0.117 -0.046 0.088 rpy=0 0 0 -> xyz=0.119 -0.046 0.088 rpy=0 0 0
- joint inkcap_right_small_0_joint: origin xyz=0.073 -0.025 0.088 rpy=0 0 0 -> xyz=0.075 -0.025 0.088 rpy=0 0 0
- joint inkcap_right_small_1_joint: origin xyz=0.089 -0.025 0.088 rpy=0 0 0 -> xyz=0.091 -0.025 0.088 rpy=0 0 0
- joint inkcap_right_small_2_joint: origin xyz=0.105 -0.025 0.088 rpy=0 0 0 -> xyz=0.107 -0.025 0.088 rpy=0 0 0
- joint inkcap_right_small_3_joint: origin xyz=0.121 -0.025 0.088 rpy=0 0 0 -> xyz=0.123 -0.025 0.088 rpy=0 0 0

Commit message: asd

File: urdf/tatbot.urdf (robot description, URDF)
Before this commit: robot tatbot, 88 links, 87 joints
Joints:
- joint inkcap_left_large_joint: origin xyz=0.099 0.046 0.088 rpy=0 0 0 -> xyz=0.099 0.046 0.080 rpy=0 0 0
- joint inkcap_left_medium_0_joint: origin xyz=0.079 0.046 0.088 rpy=0 0 0 -> xyz=0.079 0.046 0.080 rpy=0 0 0
- joint inkcap_left_medium_1_joint: origin xyz=0.119 0.046 0.088 rpy=0 0 0 -> xyz=0.119 0.046 0.080 rpy=0 0 0
- joint inkcap_left_small_0_joint: origin xyz=0.075 0.025 0.088 rpy=0 0 0 -> xyz=0.075 0.025 0.080 rpy=0 0 0
- joint inkcap_left_small_1_joint: origin xyz=0.091 0.025 0.088 rpy=0 0 0 -> xyz=0.091 0.025 0.080 rpy=0 0 0
- joint inkcap_left_small_2_joint: origin xyz=0.107 0.025 0.088 rpy=0 0 0 -> xyz=0.107 0.025 0.080 rpy=0 0 0
- joint inkcap_left_small_3_joint: origin xyz=0.123 0.025 0.088 rpy=0 0 0 -> xyz=0.123 0.025 0.080 rpy=0 0 0
- joint inkcap_right_large_joint: origin xyz=0.099 -0.046 0.088 rpy=0 0 0 -> xyz=0.099 -0.046 0.080 rpy=0 0 0
- joint inkcap_right_medium_0_joint: origin xyz=0.079 -0.046 0.088 rpy=0 0 0 -> xyz=0.079 -0.046 0.080 rpy=0 0 0
- joint inkcap_right_medium_1_joint: origin xyz=0.119 -0.046 0.088 rpy=0 0 0 -> xyz=0.119 -0.046 0.080 rpy=0 0 0
- joint inkcap_right_small_0_joint: origin xyz=0.075 -0.025 0.088 rpy=0 0 0 -> xyz=0.075 -0.025 0.080 rpy=0 0 0
- joint inkcap_right_small_1_joint: origin xyz=0.091 -0.025 0.088 rpy=0 0 0 -> xyz=0.091 -0.025 0.080 rpy=0 0 0
- joint inkcap_right_small_2_joint: origin xyz=0.107 -0.025 0.088 rpy=0 0 0 -> xyz=0.107 -0.025 0.080 rpy=0 0 0
- joint inkcap_right_small_3_joint: origin xyz=0.123 -0.025 0.088 rpy=0 0 0 -> xyz=0.123 -0.025 0.080 rpy=0 0 0

Commit message: asd

File: urdf/tatbot.urdf (robot description, URDF)
Before this commit: robot tatbot, 88 links, 87 joints
Joints:
- joint inkcap_left_large_joint: origin xyz=0.099 0.046 0.080 rpy=0 0 0 -> xyz=0.101 0.046 0.082 rpy=0 0 0
- joint inkcap_left_medium_0_joint: origin xyz=0.079 0.046 0.080 rpy=0 0 0 -> xyz=0.081 0.046 0.082 rpy=0 0 0
- joint inkcap_left_medium_1_joint: origin xyz=0.119 0.046 0.080 rpy=0 0 0 -> xyz=0.121 0.046 0.082 rpy=0 0 0
- joint inkcap_left_small_0_joint: origin xyz=0.075 0.025 0.080 rpy=0 0 0 -> xyz=0.077 0.025 0.082 rpy=0 0 0
- joint inkcap_left_small_1_joint: origin xyz=0.091 0.025 0.080 rpy=0 0 0 -> xyz=0.093 0.025 0.082 rpy=0 0 0
- joint inkcap_left_small_2_joint: origin xyz=0.107 0.025 0.080 rpy=0 0 0 -> xyz=0.109 0.025 0.082 rpy=0 0 0
- joint inkcap_left_small_3_joint: origin xyz=0.123 0.025 0.080 rpy=0 0 0 -> xyz=0.125 0.025 0.082 rpy=0 0 0
- joint inkcap_right_large_joint: origin xyz=0.099 -0.046 0.080 rpy=0 0 0 -> xyz=0.101 -0.046 0.082 rpy=0 0 0
- joint inkcap_right_medium_0_joint: origin xyz=0.079 -0.046 0.080 rpy=0 0 0 -> xyz=0.081 -0.046 0.082 rpy=0 0 0
- joint inkcap_right_medium_1_joint: origin xyz=0.119 -0.046 0.080 rpy=0 0 0 -> xyz=0.121 -0.046 0.082 rpy=0 0 0
- joint inkcap_right_small_0_joint: origin xyz=0.075 -0.025 0.080 rpy=0 0 0 -> xyz=0.077 -0.025 0.082 rpy=0 0 0
- joint inkcap_right_small_1_joint: origin xyz=0.091 -0.025 0.080 rpy=0 0 0 -> xyz=0.093 -0.025 0.082 rpy=0 0 0
- joint inkcap_right_small_2_joint: origin xyz=0.107 -0.025 0.080 rpy=0 0 0 -> xyz=0.109 -0.025 0.082 rpy=0 0 0
- joint inkcap_right_small_3_joint: origin xyz=0.123 -0.025 0.080 rpy=0 0 0 -> xyz=0.125 -0.025 0.082 rpy=0 0 0

Commit message: asd

File: urdf/tatbot.urdf (robot description, URDF)
Before this commit: robot tatbot, 88 links, 87 joints
Joints:
- joint inkcap_left_large_joint: origin xyz=0.101 0.046 0.082 rpy=0 0 0 -> xyz=0.101 0.051 0.082 rpy=0 0 0
- joint inkcap_left_medium_0_joint: origin xyz=0.081 0.046 0.082 rpy=0 0 0 -> xyz=0.081 0.051 0.082 rpy=0 0 0
- joint inkcap_left_medium_1_joint: origin xyz=0.121 0.046 0.082 rpy=0 0 0 -> xyz=0.121 0.051 0.082 rpy=0 0 0
- joint inkcap_left_small_0_joint: origin xyz=0.077 0.025 0.082 rpy=0 0 0 -> xyz=0.077 0.030 0.082 rpy=0 0 0
- joint inkcap_left_small_1_joint: origin xyz=0.093 0.025 0.082 rpy=0 0 0 -> xyz=0.093 0.030 0.082 rpy=0 0 0
- joint inkcap_left_small_2_joint: origin xyz=0.109 0.025 0.082 rpy=0 0 0 -> xyz=0.109 0.030 0.082 rpy=0 0 0
- joint inkcap_left_small_3_joint: origin xyz=0.125 0.025 0.082 rpy=0 0 0 -> xyz=0.125 0.030 0.082 rpy=0 0 0
- joint inkcap_right_large_joint: origin xyz=0.101 -0.046 0.082 rpy=0 0 0 -> xyz=0.101 -0.051 0.082 rpy=0 0 0
- joint inkcap_right_medium_0_joint: origin xyz=0.081 -0.046 0.082 rpy=0 0 0 -> xyz=0.081 -0.051 0.082 rpy=0 0 0
- joint inkcap_right_medium_1_joint: origin xyz=0.121 -0.046 0.082 rpy=0 0 0 -> xyz=0.121 -0.051 0.082 rpy=0 0 0
- joint inkcap_right_small_0_joint: origin xyz=0.077 -0.025 0.082 rpy=0 0 0 -> xyz=0.077 -0.030 0.082 rpy=0 0 0
- joint inkcap_right_small_1_joint: origin xyz=0.093 -0.025 0.082 rpy=0 0 0 -> xyz=0.093 -0.030 0.082 rpy=0 0 0
- joint inkcap_right_small_2_joint: origin xyz=0.109 -0.025 0.082 rpy=0 0 0 -> xyz=0.109 -0.030 0.082 rpy=0 0 0
- joint inkcap_right_small_3_joint: origin xyz=0.125 -0.025 0.082 rpy=0 0 0 -> xyz=0.125 -0.030 0.082 rpy=0 0 0

Commit message: asd

File: urdf/tatbot.urdf (robot description, URDF)
Before this commit: robot tatbot, 88 links, 87 joints
Joints:
- joint inkcap_left_large_joint: origin xyz=0.101 0.051 0.082 rpy=0 0 0 -> xyz=0.101 0.051 0.08 rpy=0 0 0
- joint inkcap_left_medium_0_joint: origin xyz=0.081 0.051 0.082 rpy=0 0 0 -> xyz=0.081 0.051 0.08 rpy=0 0 0
- joint inkcap_left_medium_1_joint: origin xyz=0.121 0.051 0.082 rpy=0 0 0 -> xyz=0.121 0.051 0.08 rpy=0 0 0
- joint inkcap_left_small_0_joint: origin xyz=0.077 0.030 0.082 rpy=0 0 0 -> xyz=0.077 0.030 0.08 rpy=0 0 0
- joint inkcap_left_small_1_joint: origin xyz=0.093 0.030 0.082 rpy=0 0 0 -> xyz=0.093 0.030 0.08 rpy=0 0 0
- joint inkcap_left_small_2_joint: origin xyz=0.109 0.030 0.082 rpy=0 0 0 -> xyz=0.109 0.030 0.08 rpy=0 0 0
- joint inkcap_left_small_3_joint: origin xyz=0.125 0.030 0.082 rpy=0 0 0 -> xyz=0.125 0.030 0.08 rpy=0 0 0
- joint inkcap_right_large_joint: origin xyz=0.101 -0.051 0.082 rpy=0 0 0 -> xyz=0.101 -0.051 0.08 rpy=0 0 0
- joint inkcap_right_medium_0_joint: origin xyz=0.081 -0.051 0.082 rpy=0 0 0 -> xyz=0.081 -0.051 0.08 rpy=0 0 0
- joint inkcap_right_medium_1_joint: origin xyz=0.121 -0.051 0.082 rpy=0 0 0 -> xyz=0.121 -0.051 0.08 rpy=0 0 0
- joint inkcap_right_small_0_joint: origin xyz=0.077 -0.030 0.082 rpy=0 0 0 -> xyz=0.077 -0.030 0.08 rpy=0 0 0
- joint inkcap_right_small_1_joint: origin xyz=0.093 -0.030 0.082 rpy=0 0 0 -> xyz=0.093 -0.030 0.08 rpy=0 0 0
- joint inkcap_right_small_2_joint: origin xyz=0.109 -0.030 0.082 rpy=0 0 0 -> xyz=0.109 -0.030 0.08 rpy=0 0 0
- joint inkcap_right_small_3_joint: origin xyz=0.125 -0.030 0.082 rpy=0 0 0 -> xyz=0.125 -0.030 0.08 rpy=0 0 0

Commit message: asd

File: urdf/tatbot.urdf (robot description, URDF)
Before this commit: robot tatbot, 88 links, 87 joints
Joints:
- joint inkcap_left_large_joint: origin xyz=0.101 0.051 0.08 rpy=0 0 0 -> xyz=0.101 0.053 0.08 rpy=0 0 0
- joint inkcap_left_medium_0_joint: origin xyz=0.081 0.051 0.08 rpy=0 0 0 -> xyz=0.081 0.053 0.08 rpy=0 0 0
- joint inkcap_left_medium_1_joint: origin xyz=0.121 0.051 0.08 rpy=0 0 0 -> xyz=0.121 0.053 0.08 rpy=0 0 0
- joint inkcap_left_small_0_joint: origin xyz=0.077 0.030 0.08 rpy=0 0 0 -> xyz=0.077 0.032 0.08 rpy=0 0 0
- joint inkcap_left_small_1_joint: origin xyz=0.093 0.030 0.08 rpy=0 0 0 -> xyz=0.093 0.032 0.08 rpy=0 0 0
- joint inkcap_left_small_2_joint: origin xyz=0.109 0.030 0.08 rpy=0 0 0 -> xyz=0.109 0.032 0.08 rpy=0 0 0
- joint inkcap_left_small_3_joint: origin xyz=0.125 0.030 0.08 rpy=0 0 0 -> xyz=0.125 0.032 0.08 rpy=0 0 0
- joint inkcap_right_large_joint: origin xyz=0.101 -0.051 0.08 rpy=0 0 0 -> xyz=0.101 -0.053 0.08 rpy=0 0 0
- joint inkcap_right_medium_0_joint: origin xyz=0.081 -0.051 0.08 rpy=0 0 0 -> xyz=0.081 -0.053 0.08 rpy=0 0 0
- joint inkcap_right_medium_1_joint: origin xyz=0.121 -0.051 0.08 rpy=0 0 0 -> xyz=0.121 -0.053 0.08 rpy=0 0 0
- joint inkcap_right_small_0_joint: origin xyz=0.077 -0.030 0.08 rpy=0 0 0 -> xyz=0.077 -0.032 0.08 rpy=0 0 0
- joint inkcap_right_small_1_joint: origin xyz=0.093 -0.030 0.08 rpy=0 0 0 -> xyz=0.093 -0.032 0.08 rpy=0 0 0
- joint inkcap_right_small_2_joint: origin xyz=0.109 -0.030 0.08 rpy=0 0 0 -> xyz=0.109 -0.032 0.08 rpy=0 0 0
- joint inkcap_right_small_3_joint: origin xyz=0.125 -0.030 0.08 rpy=0 0 0 -> xyz=0.125 -0.032 0.08 rpy=0 0 0

Commit message: asd

File: urdf/tatbot.urdf (robot description, URDF)
Before this commit: robot tatbot, 88 links, 87 joints
Joints:
- joint camera1_mount_joint: origin xyz=-0.0275 0.09 0.2 rpy=0 1.5707963267948966 -1.5707963267948966 -> xyz=-0.04 0 0.05 rpy=0 0 0

Commit message: origin widget

File: urdf/tatbot.urdf (robot description, URDF)
Before this commit: robot tatbot, 88 links, 87 joints
Links:
- removed link tag1
- removed link tag2
- removed link tag3
- added link origin_widget; visual mesh filename=meshes/frame/origin_widget.stl scale=0.001 0.001 0.001
- added link origin_widget_left
- added link origin_widget_right
- link tag0: geometry visual mesh filename=meshes/tags/16h5_008_4cm/tag.obj scale=1 1 1
Joints:
- removed joint tag1_joint
- removed joint tag2_joint
- removed joint tag3_joint
- added joint origin_widget_joint: type fixed, parent root, child origin_widget, origin xyz=0.152 0 0 rpy=0 0 0
- added joint origin_widget_left_joint: type fixed, parent origin_widget, child origin_widget_left, origin xyz=0 0.0375 0.003 rpy=0 0 0
- added joint origin_widget_right_joint: type fixed, parent origin_widget, child origin_widget_right, origin xyz=0 -0.0375 0.003 rpy=0 0 0
- joint tag0_joint: origin xyz=-0.02 0 0 rpy=0 0 0 -> xyz=0 0 0.0035 rpy=0 0 0; parent root -> origin_widget

Commit message: asd

File: urdf/tatbot.urdf (robot description, URDF)
Before this commit: robot tatbot, 88 links, 87 joints
Links:
- removed link palette
Joints:
- removed joint palette_joint
- joint camera1_mount_joint: origin xyz=-0.04 0 0.05 rpy=0 0 0 -> xyz=-0.2 0 0 rpy=0 0 0; parent root -> origin_widget
- joint inkcap_left_large_joint: origin xyz=0.101 0.053 0.08 rpy=0 0 0 -> xyz=-0.06 0.053 0 rpy=0 0 0; parent palette -> origin_widget
- joint inkcap_left_medium_0_joint: origin xyz=0.081 0.053 0.08 rpy=0 0 0 -> xyz=-0.080 0.053 0 rpy=0 0 0; parent palette -> origin_widget
- joint inkcap_left_medium_1_joint: origin xyz=0.121 0.053 0.08 rpy=0 0 0 -> xyz=-0.040 0.053 0 rpy=0 0 0; parent palette -> origin_widget
- joint inkcap_left_small_0_joint: origin xyz=0.077 0.032 0.08 rpy=0 0 0 -> xyz=-0.084 0.032 0 rpy=0 0 0; parent palette -> origin_widget
- joint inkcap_left_small_1_joint: origin xyz=0.093 0.032 0.08 rpy=0 0 0 -> xyz=-0.068 0.032 0 rpy=0 0 0; parent palette -> origin_widget
- joint inkcap_left_small_2_joint: origin xyz=0.109 0.032 0.08 rpy=0 0 0 -> xyz=-0.052 0.032 0 rpy=0 0 0; parent palette -> origin_widget
- joint inkcap_left_small_3_joint: origin xyz=0.125 0.032 0.08 rpy=0 0 0 -> xyz=-0.036 0.032 0 rpy=0 0 0; parent palette -> origin_widget
- joint inkcap_right_large_joint: origin xyz=0.101 -0.053 0.08 rpy=0 0 0 -> xyz=-0.06 -0.053 0 rpy=0 0 0; parent palette -> origin_widget
- joint inkcap_right_medium_0_joint: origin xyz=0.081 -0.053 0.08 rpy=0 0 0 -> xyz=-0.080 -0.053 0 rpy=0 0 0; parent palette -> origin_widget
- joint inkcap_right_medium_1_joint: origin xyz=0.121 -0.053 0.08 rpy=0 0 0 -> xyz=-0.040 -0.053 0 rpy=0 0 0; parent palette -> origin_widget
- joint inkcap_right_small_0_joint: origin xyz=0.077 -0.032 0.08 rpy=0 0 0 -> xyz=-0.084 -0.032 0 rpy=0 0 0; parent palette -> origin_widget
- joint inkcap_right_small_1_joint: origin xyz=0.093 -0.032 0.08 rpy=0 0 0 -> xyz=-0.068 -0.032 0 rpy=0 0 0; parent palette -> origin_widget
- joint inkcap_right_small_2_joint: origin xyz=0.109 -0.032 0.08 rpy=0 0 0 -> xyz=-0.052 -0.032 0 rpy=0 0 0; parent palette -> origin_widget
- joint inkcap_right_small_3_joint: origin xyz=0.125 -0.032 0.08 rpy=0 0 0 -> xyz=-0.036 -0.032 0 rpy=0 0 0; parent palette -> origin_widget
- joint origin_widget_joint: origin xyz=0.152 0 0 rpy=0 0 0 -> xyz=0.152 0 0.08 rpy=0 0 0

Commit message: asd

File: urdf/tatbot.urdf (robot description, URDF)
Before this commit: robot tatbot, 87 links, 86 joints
Joints:
- joint inkcap_left_large_joint: origin xyz=-0.06 0.053 0 rpy=0 0 0 -> xyz=-0.06 0.051 0 rpy=0 0 0
- joint inkcap_left_medium_0_joint: origin xyz=-0.080 0.053 0 rpy=0 0 0 -> xyz=-0.082 0.051 0 rpy=0 0 0
- joint inkcap_left_medium_1_joint: origin xyz=-0.040 0.053 0 rpy=0 0 0 -> xyz=-0.038 0.051 0 rpy=0 0 0
- joint inkcap_left_small_0_joint: origin xyz=-0.084 0.032 0 rpy=0 0 0 -> xyz=-0.084 0.028 0 rpy=0 0 0
- joint inkcap_left_small_1_joint: origin xyz=-0.068 0.032 0 rpy=0 0 0 -> xyz=-0.068 0.028 0 rpy=0 0 0
- joint inkcap_left_small_2_joint: origin xyz=-0.052 0.032 0 rpy=0 0 0 -> xyz=-0.052 0.028 0 rpy=0 0 0
- joint inkcap_left_small_3_joint: origin xyz=-0.036 0.032 0 rpy=0 0 0 -> xyz=-0.036 0.028 0 rpy=0 0 0
- joint inkcap_right_large_joint: origin xyz=-0.06 -0.053 0 rpy=0 0 0 -> xyz=-0.06 -0.051 0 rpy=0 0 0
- joint inkcap_right_medium_0_joint: origin xyz=-0.080 -0.053 0 rpy=0 0 0 -> xyz=-0.082 -0.051 0 rpy=0 0 0
- joint inkcap_right_medium_1_joint: origin xyz=-0.040 -0.053 0 rpy=0 0 0 -> xyz=-0.038 -0.051 0 rpy=0 0 0
- joint inkcap_right_small_0_joint: origin xyz=-0.084 -0.032 0 rpy=0 0 0 -> xyz=-0.084 -0.028 0 rpy=0 0 0
- joint inkcap_right_small_1_joint: origin xyz=-0.068 -0.032 0 rpy=0 0 0 -> xyz=-0.068 -0.028 0 rpy=0 0 0
- joint inkcap_right_small_2_joint: origin xyz=-0.052 -0.032 0 rpy=0 0 0 -> xyz=-0.052 -0.028 0 rpy=0 0 0
- joint inkcap_right_small_3_joint: origin xyz=-0.036 -0.032 0 rpy=0 0 0 -> xyz=-0.036 -0.028 0 rpy=0 0 0

Commit message: asd

File: urdf/tatbot.urdf (robot description, URDF)
Before this commit: robot tatbot, 87 links, 86 joints
Joints:
- joint origin_widget_joint: origin xyz=0.152 0 0.08 rpy=0 0 0 -> xyz=0.154 0 0.08 rpy=0 0 0
- joint origin_widget_left_joint: origin xyz=0 0.0375 0.003 rpy=0 0 0 -> xyz=0 0.0375 0.005 rpy=0 0 0
- joint origin_widget_right_joint: origin xyz=0 -0.0375 0.003 rpy=0 0 0 -> xyz=0 -0.0375 0.005 rpy=0 0 0

Commit message: asd

File: urdf/tatbot.urdf (robot description, URDF)
Before this commit: robot tatbot, 87 links, 86 joints
Joints:
- joint origin_widget_joint: origin xyz=0.154 0 0.08 rpy=0 0 0 -> xyz=0.158 0 0.08 rpy=0 0 0

Commit message: asd

File: urdf/tatbot.urdf (robot description, URDF)
Before this commit: robot tatbot, 87 links, 86 joints
Joints:
- joint origin_widget_joint: origin xyz=0.158 0 0.08 rpy=0 0 0 -> xyz=0.16 0 0.08 rpy=0 0 0

Commit message: Refactor URDF structure: renamed 'origin_widget' to 'palette', updated joint references, and removed unused components. Deleted origin_widget.stl mesh file.

File: urdf/tatbot.urdf (robot description, URDF)
Before this commit: robot tatbot, 87 links, 86 joints
Links:
- removed link inkcap_left_small_2
- removed link inkcap_left_small_3
- removed link inkcap_right_small_2
- removed link inkcap_right_small_3
- removed link origin_widget
- removed link origin_widget_left
- removed link origin_widget_right
- added link palette; visual mesh filename=meshes/frame/palette.stl scale=0.001 0.001 0.001
- added link palette_calibrator
Joints:
- removed joint inkcap_left_small_2_joint
- removed joint inkcap_left_small_3_joint
- removed joint inkcap_right_small_2_joint
- removed joint inkcap_right_small_3_joint
- removed joint origin_widget_joint
- removed joint origin_widget_left_joint
- removed joint origin_widget_right_joint
- added joint palette_calibrator_joint: type fixed, parent palette, child palette_calibrator, origin xyz=0.038 0 0.006 rpy=0 0 0
- added joint palette_joint: type fixed, parent root, child palette, origin xyz=0.16 0 0.08 rpy=0 0 0
- joint camera1_mount_joint: parent origin_widget -> palette
- joint inkcap_left_large_joint: origin xyz=-0.06 0.051 0 rpy=0 0 0 -> xyz=0 0.055 0 rpy=0 0 0; parent origin_widget -> palette
- joint inkcap_left_medium_0_joint: origin xyz=-0.082 0.051 0 rpy=0 0 0 -> xyz=0.01 0.039 0 rpy=0 0 0; parent origin_widget -> palette
- joint inkcap_left_medium_1_joint: origin xyz=-0.038 0.051 0 rpy=0 0 0 -> xyz=-0.01 0.039 0 rpy=0 0 0; parent origin_widget -> palette
- joint inkcap_left_small_0_joint: origin xyz=-0.084 0.028 0 rpy=0 0 0 -> xyz=0.008 0.069 0 rpy=0 0 0; parent origin_widget -> palette
- joint inkcap_left_small_1_joint: origin xyz=-0.068 0.028 0 rpy=0 0 0 -> xyz=-0.008 0.069 0 rpy=0 0 0; parent origin_widget -> palette
- joint inkcap_right_large_joint: origin xyz=-0.06 -0.051 0 rpy=0 0 0 -> xyz=0 -0.055 0 rpy=0 0 0; parent origin_widget -> palette
- joint inkcap_right_medium_0_joint: origin xyz=-0.082 -0.051 0 rpy=0 0 0 -> xyz=0.01 -0.039 0 rpy=0 0 0; parent origin_widget -> palette
- joint inkcap_right_medium_1_joint: origin xyz=-0.038 -0.051 0 rpy=0 0 0 -> xyz=-0.01 -0.039 0 rpy=0 0 0; parent origin_widget -> palette
- joint inkcap_right_small_0_joint: origin xyz=-0.084 -0.028 0 rpy=0 0 0 -> xyz=0.008 -0.069 0 rpy=0 0 0; parent origin_widget -> palette
- joint inkcap_right_small_1_joint: origin xyz=-0.068 -0.028 0 rpy=0 0 0 -> xyz=-0.008 -0.069 0 rpy=0 0 0; parent origin_widget -> palette
- joint tag0_joint: parent origin_widget -> palette

Commit message: asd

File: urdf/tatbot.urdf (robot description, URDF)
Before this commit: robot tatbot, 82 links, 81 joints
Joints:
- joint palette_joint: origin xyz=0.16 0 0.08 rpy=0 0 0 -> xyz=0.12 0 0.08 rpy=0 0 0

Commit message: asd

File: urdf/tatbot.urdf (robot description, URDF)
Before this commit: robot tatbot, 82 links, 81 joints
Joints:
- joint camera1_frame_joint: origin xyz=0 0 0.07 rpy=-1.5707963267948966 0 0.7853981633974483 -> xyz=0 0 0.07 rpy=-1.5707963267948966 0 1.5707963267948966
- joint camera1_optical_joint: origin xyz=0 0 0 rpy=-1.5707963267948966 0 -1.5707963267948966 -> xyz=0 0 0 rpy=-0.7853981633974483 0 -1.5707963267948966

Commit message: asd

File: urdf/tatbot.urdf (robot description, URDF)
Before this commit: robot tatbot, 82 links, 81 joints
Joints:
- joint camera1_frame_joint: origin xyz=0 0 0.07 rpy=-1.5707963267948966 0 1.5707963267948966 -> xyz=0 0 0.07 rpy=-1.5707963267948966 0 0
- joint camera1_optical_joint: origin xyz=0 0 0 rpy=-0.7853981633974483 0 -1.5707963267948966 -> xyz=0 0 0 rpy=-1.5707963267948966 0 -0.7853981633974483

Commit message: asd

File: urdf/tatbot.urdf (robot description, URDF)
Before this commit: robot tatbot, 82 links, 81 joints
Joints:
- joint camera1_optical_joint: origin xyz=0 0 0 rpy=-1.5707963267948966 0 -0.7853981633974483 -> xyz=0 0 0 rpy=-1.5707963267948966 1.5707963267948966 -0.7853981633974483

Commit message: asd

File: urdf/tatbot.urdf (robot description, URDF)
Before this commit: robot tatbot, 82 links, 81 joints
Joints:
- joint palette_joint: origin xyz=0.12 0 0.08 rpy=0 0 0 -> xyz=0.13 0 0.09 rpy=0 0 0

Commit message: asd

File: urdf/tatbot.urdf (robot description, URDF)
Before this commit: robot tatbot, 82 links, 81 joints
Joints:
- joint palette_joint: origin xyz=0.13 0 0.09 rpy=0 0 0 -> xyz=0.125 0 0.09 rpy=0 0 0

Commit message: asd

File: urdf/tatbot.urdf (robot description, URDF)
Before this commit: robot tatbot, 82 links, 81 joints
Joints:
- joint palette_joint: origin xyz=0.125 0 0.09 rpy=0 0 0 -> xyz=0.125 0 0.085 rpy=0 0 0

Commit message: asd

File: urdf/tatbot.urdf (robot description, URDF)
Before this commit: robot tatbot, 82 links, 81 joints
Joints:
- joint palette_joint: origin xyz=0.125 0 0.085 rpy=0 0 0 -> xyz=0.126 0 0.085 rpy=0 0 0

Commit message: ik improvement

File: urdf/tatbot.urdf (robot description, URDF)
Before this commit: robot tatbot, 82 links, 81 joints
Joints:
- joint left/left_carriage_joint: limit lower=0.0 upper=0.044 effort=400.0 velocity=0.0875 -> lower=0.0 upper=0.04 effort=200.0 velocity=0.25
- joint right/right_carriage_joint: limit lower=0.0 upper=0.044 effort=400.0 velocity=0.0875 -> lower=0.0 upper=0.04 effort=200.0 velocity=0.25
