Commit message: lasercross

File: urdf/tatbot.urdf (robot description, URDF)
Before this commit: robot tatbot, 82 links, 81 joints
Links:
- added link lasercross
Joints:
- added joint lasercross_joint: type fixed, parent root, child lasercross, origin xyz=0.22 0 0.08 rpy=-1.5707963267948966 0 0

Commit message: betteah

File: urdf/tatbot.urdf (robot description, URDF)
Before this commit: robot tatbot, 83 links, 82 joints
Joints:
- joint lasercross_joint: origin xyz=0.22 0 0.08 rpy=-1.5707963267948966 0 0 -> xyz=0.22 0 0.08 rpy=0 0 0

Commit message: ee relative frames

File: urdf/tatbot.urdf (robot description, URDF)
Before this commit: robot tatbot, 83 links, 82 joints
Links:
- removed link palette
- added link palette_root; visual mesh filename=meshes/frame/palette.stl scale=0.001 0.001 0.001
Joints:
- removed joint palette_joint
- added joint palette_root_joint: type fixed, parent root, child palette_root, origin xyz=0.126 0 0.085 rpy=0 0 0
- joint camera1_mount_joint: parent palette -> palette_root
- joint inkcap_left_large_joint: parent palette -> palette_root
- joint inkcap_left_medium_0_joint: parent palette -> palette_root
- joint inkcap_left_medium_1_joint: parent palette -> palette_root
- joint inkcap_left_small_0_joint: parent palette -> palette_root
- joint inkcap_left_small_1_joint: parent palette -> palette_root
- joint inkcap_right_large_joint: parent palette -> palette_root
- joint inkcap_right_medium_0_joint: parent palette -> palette_root
- joint inkcap_right_medium_1_joint: parent palette -> palette_root
- joint inkcap_right_small_0_joint: parent palette -> palette_root
- joint inkcap_right_small_1_joint: parent palette -> palette_root
- joint lasercross_joint: origin xyz=0.22 0 0.08 rpy=0 0 0 -> xyz=0.2199999988079071 -2.7755582233073814e-18 0.07999999821186066 rpy=1.500268805451172e-17 0.3897078645738488 -0.37438698854230174
- joint palette_calibrator_joint: parent palette -> palette_root
- joint tag0_joint: parent palette -> palette_root

Commit message: asd

File: urdf/tatbot.urdf (robot description, URDF)
Before this commit: robot tatbot, 83 links, 82 joints
Joints:
- joint lasercross_joint: origin xyz=0.2199999988079071 -2.7755582233073814e-18 0.07999999821186066 rpy=1.500268805451172e-17 0.3897078645738488 -0.37438698854230174 -> xyz=0.22 0 0.08 rpy=0 0 0

Commit message: align to table, paper with pen ees

File: urdf/tatbot.urdf (robot description, URDF)
Before this commit: robot tatbot, 83 links, 82 joints
Joints:
- joint lasercross_joint: origin xyz=0.22 0 0.08 rpy=0 0 0 -> xyz=0.209010 0.00 0.106720 rpy=0.000000 0.000000 0.000000

Commit message: adjustments

File: urdf/tatbot.urdf (robot description, URDF)
Before this commit: robot tatbot, 83 links, 82 joints
Joints:
- joint lasercross_joint: origin xyz=0.209010 0.00 0.106720 rpy=0.000000 0.000000 0.000000 -> xyz=0.209010 0.00 0.105 rpy=0.000000 0.000000 0.000000

Commit message: calib for koi

File: urdf/tatbot.urdf (robot description, URDF)
Before this commit: robot tatbot, 83 links, 82 joints
Joints:
- joint lasercross_joint: origin xyz=0.209010 0.00 0.105 rpy=0.000000 0.000000 0.000000 -> xyz=0.250450 0.000000 0.035928 rpy=0.000000 0.000000 0.000000

Commit message: asd

File: urdf/tatbot.urdf (robot description, URDF)
Before this commit: robot tatbot, 83 links, 82 joints
Joints:
- joint lasercross_joint: origin xyz=0.250450 0.000000 0.035928 rpy=0.000000 0.000000 0.000000 -> xyz=0.250450 0.000000 0.036 rpy=0.000000 0.000000 0.000000

Commit message: up

File: urdf/tatbot.urdf (robot description, URDF)
Before this commit: robot tatbot, 83 links, 82 joints
Joints:
- joint lasercross_joint: origin xyz=0.250450 0.000000 0.036 rpy=0.000000 0.000000 0.000000 -> xyz=0.250450 0.000000 0.038 rpy=0.000000 0.000000 0.000000

Commit message: v4 ee in urdf

File: urdf/tatbot.urdf (robot description, URDF)
Before this commit: robot tatbot, 83 links, 82 joints
Links:
- removed link left/ee_p1
- removed link left/ee_p2
- removed link right/ee_p1
- removed link right/ee_p2
- added link left/ee; visual mesh filename=meshes/ee/v4.stl scale=1 1 1
- added link right/ee; visual mesh filename=meshes/ee/v4.stl scale=1 1 1
Joints:
- removed joint left/ee_p1_joint
- removed joint left/ee_p2_joint
- removed joint right/ee_p1_joint
- removed joint right/ee_p2_joint
- added joint left/ee_joint: type fixed, parent left/carriage_left, child left/ee, origin xyz=0 0 0 rpy=0 0 0
- added joint right/ee_joint: type fixed, parent right/carriage_right, child right/ee, origin xyz=0 0 0 rpy=0 0 0
- joint left/tattoo_pen_joint: origin xyz=0.051 0.051 0 rpy=-1.5707963267948966 0 0.7853981633974483 -> xyz=0.05 0 0 rpy=0 -1.5707963267948966 0; parent left/ee_p1 -> left/ee
- joint right/tattoo_pen_joint: origin xyz=0.051 -0.051 0 rpy=1.5707963267948966 0 -0.7853981633974483 -> xyz=0.05 0 0 rpy=0 -1.5707963267948966 0; parent right/ee_p1 -> right/ee

Commit message: asd

File: urdf/tatbot.urdf (robot description, URDF)
Before this commit: robot tatbot, 81 links, 80 joints
Joints:
- joint lasercross_joint: origin xyz=0.250450 0.000000 0.038 rpy=0.000000 0.000000 0.000000 -> xyz=0.33 0.000000 0.038 rpy=0.000000 0.000000 0.000000

Commit message: asd

File: urdf/tatbot.urdf (robot description, URDF)
Before this commit: robot tatbot, 81 links, 80 joints
Joints:
- joint left/left_carriage_joint: limit lower=0.0 upper=0.04 effort=200.0 velocity=0.25 -> lower=0.0 upper=0.01 effort=200.0 velocity=0.25
- joint right/right_carriage_joint: limit lower=0.0 upper=0.04 effort=200.0 velocity=0.25 -> lower=0.0 upper=0.01 effort=200.0 velocity=0.25

Commit message: asd

File: urdf/tatbot.urdf (robot description, URDF)
Before this commit: robot tatbot, 81 links, 80 joints
Joints:
- joint lasercross_joint: origin xyz=0.33 0.000000 0.038 rpy=0.000000 0.000000 0.000000 -> xyz=0.33 0.000000 0.038 rpy=0.0 0.0 -1.5707963267948966

Commit message: asd

File: urdf/tatbot.urdf (robot description, URDF)
Before this commit: robot tatbot, 81 links, 80 joints
Joints:
- joint lasercross_joint: origin xyz=0.33 0.000000 0.038 rpy=0.0 0.0 -1.5707963267948966 -> xyz=0.33 0.000000 0.04 rpy=0.0 0.0 -1.5707963267948966

Commit message: rever eev4 back to eev3

File: urdf/tatbot.urdf (robot description, URDF)
Before this commit: robot tatbot, 81 links, 80 joints
Links:
- removed link left/ee
- removed link right/ee
- added link left/ee_p1; visual mesh filename=meshes/ee/p1.stl scale=0.001 0.001 0.001
- added link left/ee_p2; visual mesh filename=meshes/ee/p2.stl scale=0.001 0.001 0.001
- added link right/ee_p1; visual mesh filename=meshes/ee/p1.stl scale=0.001 0.001 0.001
- added link right/ee_p2; visual mesh filename=meshes/ee/p2.stl scale=0.001 0.001 0.001
Joints:
- removed joint left/ee_joint
- removed joint right/ee_joint
- added joint left/ee_p1_joint: type fixed, parent left/carriage_left, child left/ee_p1, origin xyz=0 0 0 rpy=0 0 0
- added joint left/ee_p2_joint: type fixed, parent left/ee_p1, child left/ee_p2, origin xyz=0 0 0 rpy=0 0 0
- added joint right/ee_p1_joint: type fixed, parent right/carriage_right, child right/ee_p1, origin xyz=0 0 0 rpy=0 0 0
- added joint right/ee_p2_joint: type fixed, parent right/ee_p1, child right/ee_p2, origin xyz=0 0 0 rpy=0 0 0
- joint lasercross_joint: origin xyz=0.33 0.000000 0.04 rpy=0.0 0.0 -1.5707963267948966 -> xyz=0.250450 0.000000 0.038 rpy=0.000000 0.000000 0.000000
- joint left/left_carriage_joint: limit lower=0.0 upper=0.01 effort=200.0 velocity=0.25 -> lower=0.0 upper=0.04 effort=200.0 velocity=0.25
- joint left/tattoo_pen_joint: origin xyz=0.05 0 0 rpy=0 -1.5707963267948966 0 -> xyz=0.051 0.051 0 rpy=-1.5707963267948966 0 0.7853981633974483; parent left/ee -> left/ee_p1
- joint right/right_carriage_joint: limit lower=0.0 upper=0.01 effort=200.0 velocity=0.25 -> lower=0.0 upper=0.04 effort=200.0 velocity=0.25
- joint right/tattoo_pen_joint: origin xyz=0.05 0 0 rpy=0 -1.5707963267948966 0 -> xyz=0.051 -0.051 0 rpy=1.5707963267948966 0 -0.7853981633974483; parent right/ee -> right/ee_p1

Commit message: asd

File: urdf/tatbot.urdf (robot description, URDF)
Before this commit: robot tatbot, 83 links, 82 joints
Joints:
- joint lasercross_joint: origin xyz=0.250450 0.000000 0.038 rpy=0.000000 0.000000 0.000000 -> xyz=0.250450 0.000000 0.03 rpy=0.000000 0.000000 0.000000

Commit message: tune

File: urdf/tatbot.urdf (robot description, URDF)
Before this commit: robot tatbot, 83 links, 82 joints
Joints:
- joint lasercross_joint: origin xyz=0.250450 0.000000 0.03 rpy=0.000000 0.000000 0.000000 -> xyz=0.250450 0.000000 0.028 rpy=0.000000 0.000000 0.000000

Commit message: fake arm

File: urdf/tatbot.urdf (robot description, URDF)
Before this commit: robot tatbot, 83 links, 82 joints
Joints:
- joint lasercross_joint: origin xyz=0.250450 0.000000 0.028 rpy=0.000000 0.000000 0.000000 -> xyz=0.250450 0.000000 0.1 rpy=0.000000 0.000000 0.000000

Commit message: calib

File: urdf/tatbot.urdf (robot description, URDF)
Before this commit: robot tatbot, 83 links, 82 joints
Joints:
- joint lasercross_joint: origin xyz=0.250450 0.000000 0.1 rpy=0.000000 0.000000 0.000000 -> xyz=0.250450 0.000000 0.125 rpy=0.000000 0.000000 0.000000

Commit message: fix: update frame construction in align and stroke tools; modify URDF to toggle fake arm visibility

File: urdf/tatbot.urdf (robot description, URDF)
Before this commit: robot tatbot, 83 links, 82 joints
Joints:
- joint lasercross_joint: origin xyz=0.250450 0.000000 0.125 rpy=0.000000 0.000000 0.000000 -> xyz=0.250450 0.000000 0.028 rpy=0.000000 0.000000 0.000000

Commit message: arm demo

File: urdf/tatbot.urdf (robot description, URDF)
Before this commit: robot tatbot, 83 links, 82 joints
Joints:
- joint lasercross_joint: origin xyz=0.250450 0.000000 0.028 rpy=0.000000 0.000000 0.000000 -> xyz=0.250450 0.000000 0.14 rpy=0.000000 0.000000 -1.5707963267948966

Commit message: asd

File: urdf/tatbot.urdf (robot description, URDF)
Before this commit: robot tatbot, 83 links, 82 joints
Joints:
- joint lasercross_joint: origin xyz=0.250450 0.000000 0.14 rpy=0.000000 0.000000 -1.5707963267948966 -> xyz=0.250450 0.000000 0.88 rpy=0.000000 0.000000 -1.5707963267948966

Commit message: tune

File: urdf/tatbot.urdf (robot description, URDF)
Before this commit: robot tatbot, 83 links, 82 joints
Joints:
- joint lasercross_joint: origin xyz=0.250450 0.000000 0.88 rpy=0.000000 0.000000 -1.5707963267948966 -> xyz=0.250450 0.000000 0.09 rpy=0.000000 0.000000 -1.5707963267948966

Commit message: tune

File: urdf/tatbot.urdf (robot description, URDF)
Before this commit: robot tatbot, 83 links, 82 joints
Joints:
- joint lasercross_joint: origin xyz=0.250450 0.000000 0.09 rpy=0.000000 0.000000 -1.5707963267948966 -> xyz=0.250450 0.000000 0.108 rpy=0.000000 0.000000 -1.5707963267948966

Commit message: tune

File: urdf/tatbot.urdf (robot description, URDF)
Before this commit: robot tatbot, 83 links, 82 joints
Joints:
- joint lasercross_joint: origin xyz=0.250450 0.000000 0.108 rpy=0.000000 0.000000 -1.5707963267948966 -> xyz=0.250450 0.000000 0.10 rpy=0.000000 0.000000 0.000000

Commit message: tune

File: urdf/tatbot.urdf (robot description, URDF)
Before this commit: robot tatbot, 83 links, 82 joints
Joints:
- joint lasercross_joint: origin xyz=0.250450 0.000000 0.10 rpy=0.000000 0.000000 0.000000 -> xyz=0.250450 0.000000 0.108 rpy=0.000000 0.000000 0.000000

Commit message: tune

File: urdf/tatbot.urdf (robot description, URDF)
Before this commit: robot tatbot, 83 links, 82 joints
Joints:
- joint lasercross_joint: origin xyz=0.250450 0.000000 0.108 rpy=0.000000 0.000000 0.000000 -> xyz=0.250450 0.000000 0.102 rpy=0.000000 0.000000 0.000000
