Commit message: export 20260902
source: e47f976cebbc8a55ead1da6d45980f0ecbd586c8

manifest: cd63945d01e6cbe18db660df72e199666fd6a760f226dae808f4930a908d5a5a

File: urdf/tatbot.urdf (robot description, URDF)
Before this commit: robot tatbot, 89 links, 88 joints
Links:
- link right/tattoo_needle: geometry collision sphere radius=0.00025
Joints:
- joint right/tattoo_needle_joint: origin xyz=0 0 0.0694479075 rpy=0 0 0 -> xyz=0 0 0.06 rpy=0 0 0
- joint right/tattoo_pen_joint: origin xyz=0 0 0 rpy=0 0.162855098 1.70351218 -> xyz=-0.000202704196 0.00151837686 0.00932289653 rpy=0 0.162855098 1.70351218

Commit message: export 0.10.0
source: 42e17925603589568b456c93b45b143a00cd6b27

File: urdf/tatbot.urdf (robot description, URDF)
Before this commit: robot tatbot, 89 links, 88 joints
Links:
- removed link inkcap_left_large
- removed link inkcap_left_medium_0
- removed link inkcap_left_medium_1
- removed link inkcap_left_small_0
- removed link inkcap_left_small_1
- removed link inkcap_right_large
- removed link inkcap_right_medium_0
- removed link inkcap_right_medium_1
- removed link inkcap_right_small_0
- removed link inkcap_right_small_1
- removed link palette_calibrator
- removed link palette_root
- removed link palette_tag8
- removed link right/realsense_lower_bottom_screw_frame
- removed link right/realsense_lower_color_frame
- removed link right/realsense_lower_color_optical_frame
- removed link right/realsense_lower_depth_frame
- removed link right/realsense_lower_depth_optical_frame
- removed link right/realsense_lower_infra1_frame
- removed link right/realsense_lower_infra1_optical_frame
- removed link right/realsense_lower_infra2_frame
- removed link right/realsense_lower_infra2_optical_frame
- removed link right/realsense_lower_link
- removed link right/realsense_lower_mount_d405
- removed link right/wrist_tag6
- removed link right/wrist_tag7
- removed link right/wrist_tag8
- added link left/ee_mount; visual mesh filename=meshes/ee/fiducial-cubes-47mm-rear/left_fiducial_cube_47mm.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 scale=0.001 0.001 0.001; visual mesh filename=meshes/ee/leader-laser-v5/01_leader_cradle.stl scale=0.001 0.001 0.001
- added link left/realsense_bottom_screw_frame
- added link left/realsense_color_frame
- added link left/realsense_color_optical_frame
- added link left/realsense_depth_frame
- added link left/realsense_depth_optical_frame
- added link left/realsense_infra1_frame
- added link left/realsense_infra1_optical_frame
- added link left/realsense_infra2_frame
- added link left/realsense_infra2_optical_frame
- added link left/realsense_link, mass 0.072; collision box size=0.023 0.042 0.042; visual mesh filename=meshes/cameras/d405.stl scale=0.001 0.001 0.001
- added link left/realsense_mount_d405, mass 0.04518012; collision mesh filename=meshes/wxai/camera_mount_d405.stl; visual mesh filename=meshes/wxai/camera_mount_d405.stl
- added link left/tattoo_needle
- added link left/tattoo_pen; visual cylinder length=0.000375 radius=0.018803125; visual cylinder length=0.000375 radius=0.018809375
- added link left/tool_mount
- added link left/wrist_tag1; visual mesh filename=meshes/tags/36h11_001_47mm/tag.glb
- added link left/wrist_tag30; visual mesh filename=meshes/tags/36h11_030_47mm/tag.glb
- added link left/wrist_tag5; visual mesh filename=meshes/tags/36h11_005_47mm/tag.glb
- added link rig_center
- added link right/wrist_tag2; visual mesh filename=meshes/tags/36h11_002_47mm/tag.glb
- added link right/wrist_tag4; visual mesh filename=meshes/tags/36h11_004_47mm/tag.glb
- link left/handle: mass 0.05670184 -> None; geometry 
- link left/leader_finger_left_index: mass 0.02647075 -> None; geometry 
- link left/leader_finger_left_thumb: mass 0.02088075 -> None; geometry 
- link right/ee_mount: geometry visual mesh filename=meshes/ee/fiducial-cubes-47mm-rear/right_fiducial_cube_47mm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 scale=0.001 0.001 0.001; visual mesh filename=meshes/ee/v17/01_cradle_and_brace.stl scale=0.001 0.001 0.001
- link right/tattoo_needle: geometry collision sphere radius=0.0005
- link right/tattoo_pen: geometry visual cylinder length=0.00014375 radius=0.003996875; visual cylinder length=0.00014375 radius=0.004190625
- link right/wrist_tag3: geometry visual mesh filename=meshes/tags/36h11_003_47mm/tag.glb
Joints:
- removed joint inkcap_left_large_joint
- removed joint inkcap_left_medium_0_joint
- removed joint inkcap_left_medium_1_joint
- removed joint inkcap_left_small_0_joint
- removed joint inkcap_left_small_1_joint
- removed joint inkcap_right_large_joint
- removed joint inkcap_right_medium_0_joint
- removed joint inkcap_right_medium_1_joint
- removed joint inkcap_right_small_0_joint
- removed joint inkcap_right_small_1_joint
- removed joint palette_calibrator_joint
- removed joint palette_root_joint
- removed joint palette_tag8_joint
- removed joint right/realsense_lower_color_joint
- removed joint right/realsense_lower_color_optical_joint
- removed joint right/realsense_lower_depth_joint
- removed joint right/realsense_lower_depth_optical_joint
- removed joint right/realsense_lower_infra1_joint
- removed joint right/realsense_lower_infra1_optical_joint
- removed joint right/realsense_lower_infra2_joint
- removed joint right/realsense_lower_infra2_optical_joint
- removed joint right/realsense_lower_joint
- removed joint right/realsense_lower_link_joint
- removed joint right/realsense_lower_mount_joint
- removed joint right/wrist_tag6_joint
- removed joint right/wrist_tag7_joint
- removed joint right/wrist_tag8_joint
- added joint left/ee_mount_joint: type fixed, parent left/carriage_left, child left/ee_mount, origin xyz=0 0 0 rpy=3.141592653589793 0 0
- added joint left/realsense_color_joint: type fixed, parent left/realsense_link, child left/realsense_color_frame, origin xyz=0 0.0 0 rpy=0 0 0
- added joint left/realsense_color_optical_joint: type fixed, parent left/realsense_color_frame, child left/realsense_color_optical_frame, origin xyz=0 0 0 rpy=-1.5707963267948966 0 -1.5707963267948966
- added joint left/realsense_depth_joint: type fixed, parent left/realsense_link, child left/realsense_depth_frame, origin xyz=0 0 0 rpy=0 0 0
- added joint left/realsense_depth_optical_joint: type fixed, parent left/realsense_depth_frame, child left/realsense_depth_optical_frame, origin xyz=0 0 0 rpy=-1.5707963267948966 0 -1.5707963267948966
- added joint left/realsense_infra1_joint: type fixed, parent left/realsense_link, child left/realsense_infra1_frame, origin xyz=0 0.0 0 rpy=0 0 0
- added joint left/realsense_infra1_optical_joint: type fixed, parent left/realsense_infra1_frame, child left/realsense_infra1_optical_frame, origin xyz=0 0 0 rpy=-1.5707963267948966 0 -1.5707963267948966
- added joint left/realsense_infra2_joint: type fixed, parent left/realsense_link, child left/realsense_infra2_frame, origin xyz=0 -0.018 0 rpy=0 0 0
- added joint left/realsense_infra2_optical_joint: type fixed, parent left/realsense_infra2_frame, child left/realsense_infra2_optical_frame, origin xyz=0 0 0 rpy=-1.5707963267948966 0 -1.5707963267948966
- added joint left/realsense_joint: type fixed, parent left/realsense_mount_d405, child left/realsense_bottom_screw_frame, origin xyz=0.02927207801 0 0.03824951197 rpy=0 0.3490658503988659 0
- added joint left/realsense_link_joint: type fixed, parent left/realsense_bottom_screw_frame, child left/realsense_link, origin xyz=0.01085 0.009 0.021 rpy=0 0 0
- added joint left/realsense_mount_joint: type fixed, parent left/link_6, child left/realsense_mount_d405, origin xyz=0.012 0 0 rpy=0 0 0
- added joint left/tattoo_needle_joint: type fixed, parent left/tattoo_pen, child left/tattoo_needle, origin xyz=0 0 0.1395 rpy=0 0 0
- added joint left/tattoo_pen_joint: type fixed, parent left/tool_mount, child left/tattoo_pen, origin xyz=7.06798229e-05 -7.08734663e-05 0.0025552402 rpy=0 0.0391517933 -0.786766152
- added joint left/tool_mount_joint: type fixed, parent left/carriage_left, child left/tool_mount, origin xyz=0.038110806929 0.065907191271 0.000564 rpy=0.785398163397448 1.570796326794897 0
- added joint left/wrist_tag1_joint: type fixed, parent left/carriage_left, child left/wrist_tag1, origin xyz=0.06854182 0.13964242 0.02857898 rpy=-0.00164549 0.01279494 -0.01488363
- added joint left/wrist_tag30_joint: type fixed, parent left/carriage_left, child left/wrist_tag30, origin xyz=0.03075870 0.14097805 -0.00353179 rpy=-1.56511783 -0.00149562 1.55821655
- added joint left/wrist_tag5_joint: type fixed, parent left/carriage_left, child left/wrist_tag5, origin xyz=0.06941833 0.17484593 -0.00439281 rpy=-1.56956599 0.01207150 -0.02292718
- added joint rig_center_joint: type fixed, parent root, child rig_center, origin xyz=0 0 0 rpy=0 0 0
- added joint right/wrist_tag2_joint: type fixed, parent right/gripper_left, child right/wrist_tag2, origin xyz=0.06511021 0.17725353 0.00279946 rpy=-1.16134632 1.56314399 0.39138579
- added joint right/wrist_tag4_joint: type fixed, parent right/gripper_left, child right/wrist_tag4, origin xyz=0.06852751 0.14303955 -0.02861336 rpy=3.13393546 0.01172946 1.56286620
- joint 300mm_front_rail_left_joint: parent root -> rig_center
- joint 300mm_front_rail_right_joint: parent root -> rig_center
- joint 600mm_back_horizontal_joint: parent root -> rig_center
- joint 600mm_front_horizontal_joint: parent root -> rig_center
- joint 600mm_vertical_left_joint: parent root -> rig_center
- joint 600mm_vertical_right_joint: parent root -> rig_center
- joint 600mm_vertical_top_joint: parent root -> rig_center
- joint camera1_mount_joint: origin xyz=-0.2 0 0 rpy=0 0 0 -> xyz=-0.074 0 0.085 rpy=0 0 0; parent palette_root -> rig_center
- joint camera2_mount_joint: parent root -> rig_center
- joint camera3_mount_joint: parent root -> rig_center
- joint camera4_mount_joint: parent root -> rig_center
- joint camera5_mount_joint: parent root -> rig_center
- joint right/tattoo_needle_joint: origin xyz=0 0 0.06 rpy=0 0 0 -> xyz=0 0 0.073 rpy=0 0 0
- joint right/tattoo_pen_joint: origin xyz=-0.000202704196 0.00151837686 0.00932289653 rpy=0 0.162855098 1.70351218 -> xyz=-1.22733305e-05 -0.000169732368 0.00181409078 rpy=0 0.0935338947 -1.64298059
- joint right/tool_mount_joint: origin xyz=0.078444 0.044183 0 rpy=2.356194 -1.570796 0 -> xyz=0.0639202049734 0.0400977950266 -0.000564 rpy=2.356194490192345 -1.570796326794897 0
- joint right/wrist_tag3_joint: origin xyz=0.04260701 0.11760005 -0.04011157 rpy=-3.12270922 -0.01142015 1.56903879 -> xyz=0.03006740 0.14215985 0.00518638 rpy=-1.56601669 -0.00691598 1.56466469

Commit message: export 0.11.0
source: 9d7767b8d4a6948a0ffb5eb4feec23a5721c5af3

File: urdf/tatbot.urdf (robot description, URDF)
Before this commit: robot tatbot, 83 links, 82 joints
Links:
- removed link left/base_link
- removed link left/carriage_left
- removed link left/carriage_right
- removed link left/ee_gripper_link
- removed link left/ee_mount
- removed link left/handle
- removed link left/leader_finger_left_index
- removed link left/leader_finger_left_thumb
- removed link left/link_1
- removed link left/link_2
- removed link left/link_3
- removed link left/link_4
- removed link left/link_5
- removed link left/link_6
- removed link left/realsense_bottom_screw_frame
- removed link left/realsense_color_frame
- removed link left/realsense_color_optical_frame
- removed link left/realsense_depth_frame
- removed link left/realsense_depth_optical_frame
- removed link left/realsense_infra1_frame
- removed link left/realsense_infra1_optical_frame
- removed link left/realsense_infra2_frame
- removed link left/realsense_infra2_optical_frame
- removed link left/realsense_link
- removed link left/realsense_mount_d405
- removed link left/tattoo_needle
- removed link left/tattoo_pen
- removed link left/tool_mount
- removed link left/wrist_tag1
- removed link left/wrist_tag30
- removed link left/wrist_tag5
- added link right/realsense_lower_bottom_screw_frame
- added link right/realsense_lower_color_frame
- added link right/realsense_lower_color_optical_frame
- added link right/realsense_lower_depth_frame
- added link right/realsense_lower_depth_optical_frame
- added link right/realsense_lower_infra1_frame
- added link right/realsense_lower_infra1_optical_frame
- added link right/realsense_lower_infra2_frame
- added link right/realsense_lower_infra2_optical_frame
- added link right/realsense_lower_link, mass 0.072; collision box size=0.023 0.042 0.042; visual mesh filename=meshes/cameras/d405.stl scale=0.001 0.001 0.001
- added link right/realsense_lower_mount_d405, mass 0.04518012; collision mesh filename=meshes/wxai/camera_mount_d405.stl; visual mesh filename=meshes/wxai/camera_mount_d405.stl
Joints:
- removed joint left/ee_gripper
- removed joint left/ee_mount_joint
- removed joint left/handle_joint
- removed joint left/joint_0
- removed joint left/joint_1
- removed joint left/joint_2
- removed joint left/joint_3
- removed joint left/joint_4
- removed joint left/joint_5
- removed joint left/left_carriage_joint
- removed joint left/left_index_joint
- removed joint left/left_thumb_joint
- removed joint left/mount_joint
- removed joint left/realsense_color_joint
- removed joint left/realsense_color_optical_joint
- removed joint left/realsense_depth_joint
- removed joint left/realsense_depth_optical_joint
- removed joint left/realsense_infra1_joint
- removed joint left/realsense_infra1_optical_joint
- removed joint left/realsense_infra2_joint
- removed joint left/realsense_infra2_optical_joint
- removed joint left/realsense_joint
- removed joint left/realsense_link_joint
- removed joint left/realsense_mount_joint
- removed joint left/right_carriage_joint
- removed joint left/tattoo_needle_joint
- removed joint left/tattoo_pen_joint
- removed joint left/tool_mount_joint
- removed joint left/wrist_tag1_joint
- removed joint left/wrist_tag30_joint
- removed joint left/wrist_tag5_joint
- added joint right/realsense_lower_color_joint: type fixed, parent right/realsense_lower_link, child right/realsense_lower_color_frame, origin xyz=0 0.0 0 rpy=0 0 0
- added joint right/realsense_lower_color_optical_joint: type fixed, parent right/realsense_lower_color_frame, child right/realsense_lower_color_optical_frame, origin xyz=0 0 0 rpy=-1.5707963267948966 0 -1.5707963267948966
- added joint right/realsense_lower_depth_joint: type fixed, parent right/realsense_lower_link, child right/realsense_lower_depth_frame, origin xyz=0 0 0 rpy=0 0 0
- added joint right/realsense_lower_depth_optical_joint: type fixed, parent right/realsense_lower_depth_frame, child right/realsense_lower_depth_optical_frame, origin xyz=0 0 0 rpy=-1.5707963267948966 0 -1.5707963267948966
- added joint right/realsense_lower_infra1_joint: type fixed, parent right/realsense_lower_link, child right/realsense_lower_infra1_frame, origin xyz=0 0.0 0 rpy=0 0 0
- added joint right/realsense_lower_infra1_optical_joint: type fixed, parent right/realsense_lower_infra1_frame, child right/realsense_lower_infra1_optical_frame, origin xyz=0 0 0 rpy=-1.5707963267948966 0 -1.5707963267948966
- added joint right/realsense_lower_infra2_joint: type fixed, parent right/realsense_lower_link, child right/realsense_lower_infra2_frame, origin xyz=0 -0.018 0 rpy=0 0 0
- added joint right/realsense_lower_infra2_optical_joint: type fixed, parent right/realsense_lower_infra2_frame, child right/realsense_lower_infra2_optical_frame, origin xyz=0 0 0 rpy=-1.5707963267948966 0 -1.5707963267948966
- added joint right/realsense_lower_joint: type fixed, parent right/realsense_lower_mount_d405, child right/realsense_lower_bottom_screw_frame, origin xyz=0.02927207801 0 0.03824951197 rpy=0 0.3490658503988659 0
- added joint right/realsense_lower_link_joint: type fixed, parent right/realsense_lower_bottom_screw_frame, child right/realsense_lower_link, origin xyz=0.01085 0.009 0.021 rpy=0 0 0
- added joint right/realsense_lower_mount_joint: type fixed, parent right/link_6, child right/realsense_lower_mount_d405, origin xyz=0.01287 0.00091 0.0015 rpy=-3.12656 0.02674 -0.00122
- joint right/tattoo_pen_joint: origin xyz=-1.22733305e-05 -0.000169732368 0.00181409078 rpy=0 0.0935338947 -1.64298059 -> xyz=-1.43536644e-05 -0.000464332396 -0.0107529699 rpy=0 0.0431755603 1.53989369
